File: Vendo_main_board/Vendo_main_board/IO_EXPANDER.kicad_sch (KiCad schematic)
At the start: 15 parts, among them U19 MCP23017_SO

Commit message: -update scheme and pcb placement
update scheme and footprint
added spade connectors
Parts:
- JP4: renamed from JP5; footprint (none) -> Jumper:SolderJumper-2_P1.3mm_Open_RoundedPad1.0x1.5mm
- JP5: renamed from JP4; footprint (none) -> Jumper:SolderJumper-2_P1.3mm_Open_RoundedPad1.0x1.5mm
- JP6: renamed from JP3; footprint (none) -> Jumper:SolderJumper-2_P1.3mm_Open_RoundedPad1.0x1.5mm
- R17: renamed from R5; footprint Resistor_SMD:R_0402_1005Metric_Pad0.72x0.64mm_HandSolder -> Resistor_SMD:R_0603_1608Metric_Pad0.98x0.95mm_HandSolder
- R18: renamed from R6; footprint Resistor_SMD:R_0402_1005Metric_Pad0.72x0.64mm_HandSolder -> Resistor_SMD:R_0603_1608Metric_Pad0.98x0.95mm_HandSolder
- renumbered C36 to C29, C35 to C30, C34 to C31, R49 to R14, R50 to R15, R51 to R16, R53 to R19, R52 to R20, R54 to R21, U19 to U9
