File: Vendo_main_board/Vendo_main_board/NON_ISO_5V_BUCK.kicad_sch (KiCad schematic)
At the start: 15 parts, among them U12 AP64350SP-13

Commit message: -update schematic
-recheck lcsc part number ,value
-check and update footprint assignment
-add load switch for the wdt and ldo combination

-add link for quick connect footprint must be discuss for clarification
Parts:
- L2: footprint Footprint Library:744325550 -> InnovKits:744325550
- U12: footprint Footprint Library:AP64350SP-13-L -> InnovKits:AP64350SP-13-L
Changed lines of the file:
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@@
 			)
 		)
-		(property "Footprint" "Footprint Library:744325550"
+		(property "Footprint" "InnovKits:744325550"
 			(at 172.3632 78.0564 0)
 			(effects
@@
 			)
 		)
-		(property "Footprint" "Footprint Library:AP64350SP-13-L"
+		(property "Footprint" "InnovKits:AP64350SP-13-L"
 			(at 132.9094 72.0766 0)
 			(effects

Commit message: -update scheme and pcb placement
update scheme and footprint
added spade connectors
Parts:
- renumbered C19 to C1, C19 to C2, C20 to C3, C20 to C4, C31 to C5, C32 to C6, C33 to C7, L2 to L1, R44 to R1, R45 to R2, R46 to R3, R47 to R4, R48 to R5, U12 to U1
Changed lines of the file:
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@@
 		(dnp no)
 		(fields_autoplaced yes)
-		(property "Reference" "L2"
+		(property "Reference" "L1"
 			(at 172.3632 73.2136 0)
 			(effects
@@
 			(project "Vendo_main_board"
 				(path "/ce68e045-3b24-4b1f-b4c3-20bce3f1de80/4e895ab7-4f43-4499-a6a7-69405199c565"
-					(reference "L2")
+					(reference "L1")
 					(unit 1)
 				)
@@
 		(dnp no)
 		(fields_autoplaced yes)
-		(property "Reference" "C19"
+		(property "Reference" "C1"
 			(at 88.5685 83.6879 0)
 			(effects
@@
 			(project "Vendo_main_board"
 				(path "/ce68e045-3b24-4b1f-b4c3-20bce3f1de80/4e895ab7-4f43-4499-a6a7-69405199c565"
-					(reference "C19")
+					(reference "C1")
 					(unit 1)
 				)
@@
 		(dnp no)
 		(fields_autoplaced yes)
-		(property "Reference" "C32"
+		(property "Reference" "C6"
 			(at 194.5291 81.0317 0)
 			(effects
@@
 			(project "Vendo_main_board"
 				(path "/ce68e045-3b24-4b1f-b4c3-20bce3f1de80/4e895ab7-4f43-4499-a6a7-69405199c565"
-					(reference "C32")
+					(reference "C6")
 					(unit 1)
 				)
@@
 		(dnp no)
 		(fields_autoplaced yes)
-		(property "Reference" "R47"
+		(property "Reference" "R4"
 			(at 202.0238 94.8627 0)
 			(effects
@@
 			(project "Vendo_main_board"
 				(path "/ce68e045-3b24-4b1f-b4c3-20bce3f1de80/4e895ab7-4f43-4499-a6a7-69405199c565"
-					(reference "R47")
+					(reference "R4")
 					(unit 1)
 				)
@@
 		(dnp no)
 		(fields_autoplaced yes)
-		(property "Reference" "U12"
+		(property "Reference" "U1"
 			(at 132.9094 68.945 0)
 			(effects
@@
 			(project "Vendo_main_board"
 				(path "/ce68e045-3b24-4b1f-b4c3-20bce3f1de80/4e895ab7-4f43-4499-a6a7-69405199c565"
-					(reference "U12")
+					(reference "U1")
 					(unit 1)
 				)
@@
 		(dnp no)
 		(fields_autoplaced yes)
-		(property "Reference" "R44"
+		(property "Reference" "R1"
 			(at 106.8175 89.3532 0)
 			(effects
@@
 			(project "Vendo_main_board"
 				(path "/ce68e045-3b24-4b1f-b4c3-20bce3f1de80/4e895ab7-4f43-4499-a6a7-69405199c565"
-					(reference "R44")
+					(reference "R1")
 					(unit 1)
 				)
@@
 		(dnp no)
 		(fields_autoplaced yes)
-		(property "Reference" "#PWR098"
+		(property "Reference" "#PWR04"
 			(at 85.6475 109.1478 0)
 			(effects
@@
 			(project "Vendo_main_board"
 				(path "/ce68e045-3b24-4b1f-b4c3-20bce3f1de80/4e895ab7-4f43-4499-a6a7-69405199c565"
-					(reference "#PWR098")
+					(reference "#PWR04")
 					(unit 1)
 				)
@@
 		(dnp no)
 		(fields_autoplaced yes)
-		(property "Reference" "R48"
+		(property "Reference" "R5"
 			(at 229.4104 82.9355 0)
 			(effects
@@
 			(project "Vendo_main_board"
 				(path "/ce68e045-3b24-4b1f-b4c3-20bce3f1de80/4e895ab7-4f43-4499-a6a7-69405199c565"
-					(reference "R48")
+					(reference "R5")
 					(unit 1)
 				)
@@
 		(dnp no)
 		(fields_autoplaced yes)
-		(property "Reference" "#PWR061"
+		(property "Reference" "#PWR07"
 			(at 164.0362 122.6066 0)
 			(effects
@@
 			(project "Vendo_main_board"
 				(path "/ce68e045-3b24-4b1f-b4c3-20bce3f1de80/4e895ab7-4f43-4499-a6a7-69405199c565"
-					(reference "#PWR061")
+					(reference "#PWR07")
 					(unit 1)
 				)
@@
 		(dnp no)
 		(fields_autoplaced yes)
-		(property "Reference" "#PWR059"
+		(property "Reference" "#PWR09"
 			(at 184.51 123.1067 0)
 			(effects
@@
 			(project "Vendo_main_board"
 				(path "/ce68e045-3b24-4b1f-b4c3-20bce3f1de80/4e895ab7-4f43-4499-a6a7-69405199c565"
-					(reference "#PWR059")
+					(reference "#PWR09")
 					(unit 1)
 				)
@@
 		(dnp no)
 		(fields_autoplaced yes)
-		(property "Reference" "#PWR0103"
+		(property "Reference" "#PWR014"
 			(at 226.8704 123.9541 0)
 			(effects
@@
 			(project "Vendo_main_board"
 				(path "/ce68e045-3b24-4b1f-b4c3-20bce3f1de80/4e895ab7-4f43-4499-a6a7-69405199c565"
-					(reference "#PWR0103")
+					(reference "#PWR014")
 					(unit 1)
 				)
@@
 		(dnp no)
 		(fields_autoplaced yes)
-		(property "Reference" "#PWR057"
+		(property "Reference" "#PWR012"
 			(at 213.4323 123.8756 0)
 			(effects
@@
 			(project "Vendo_main_board"
 				(path "/ce68e045-3b24-4b1f-b4c3-20bce3f1de80/4e895ab7-4f43-4499-a6a7-69405199c565"
-					(reference "#PWR057")
+					(reference "#PWR012")
 					(unit 1)
 				)
@@
 		(on_board yes)
 		(dnp no)
-		(property "Reference" "#PWR099"
+		(property "Reference" "#PWR013"
 			(at 213.4406 77.6353 0)
 			(effects
@@
 			(project "Vendo_main_board"
 				(path "/ce68e045-3b24-4b1f-b4c3-20bce3f1de80/4e895ab7-4f43-4499-a6a7-69405199c565"
-					(reference "#PWR099")
+					(reference "#PWR013")
 					(unit 1)
 				)
@@
 		(dnp no)
 		(fields_autoplaced yes)
-		(property "Reference" "#PWR095"
+		(property "Reference" "#PWR06"
 			(at 104.9512 109.1478 0)
 			(effects
@@
 			(project "Vendo_main_board"
 				(path "/ce68e045-3b24-4b1f-b4c3-20bce3f1de80/4e895ab7-4f43-4499-a6a7-69405199c565"
-					(reference "#PWR095")
+					(reference "#PWR06")
 					(unit 1)
 				)
@@
 		(dnp no)
 		(fields_autoplaced yes)
-		(property "Reference" "#PWR097"
+		(property "Reference" "#PWR05"
 			(at 95.7298 109.1478 0)
 			(effects
@@
 			(project "Vendo_main_board"
 				(path "/ce68e045-3b24-4b1f-b4c3-20bce3f1de80/4e895ab7-4f43-4499-a6a7-69405199c565"
-					(reference "#PWR097")
+					(reference "#PWR05")
 					(unit 1)
 				)
@@
 		(dnp no)
 		(fields_autoplaced yes)
-		(property "Reference" "#PWR0100"
+		(property "Reference" "#PWR015"
 			(at 236.5884 68.2947 0)
 			(effects
@@
 			(project "Vendo_main_board"
 				(path "/ce68e045-3b24-4b1f-b4c3-20bce3f1de80/4e895ab7-4f43-4499-a6a7-69405199c565"
-					(reference "#PWR0100")
+					(reference "#PWR015")
 					(unit 1)
 				)
@@
 		(dnp no)
 		(fields_autoplaced yes)
-		(property "Reference" "#PWR058"
+		(property "Reference" "#PWR011"
 			(at 200.0497 123.8756 0)
 			(effects
@@
 			(project "Vendo_main_board"
 				(path "/ce68e045-3b24-4b1f-b4c3-20bce3f1de80/4e895ab7-4f43-4499-a6a7-69405199c565"
-					(reference "#PWR058")
+					(reference "#PWR011")
 					(unit 1)
 				)
@@
 		(dnp no)
 		(fields_autoplaced yes)
-		(property "Reference" "C33"
+		(property "Reference" "C7"
 			(at 216.3533 84.1957 0)
 			(effects
@@
 			(project "Vendo_main_board"
 				(path "/ce68e045-3b24-4b1f-b4c3-20bce3f1de80/4e895ab7-4f43-4499-a6a7-69405199c565"
-					(reference "C33")
+					(reference "C7")
 					(unit 1)
 				)
@@
 		(on_board yes)
 		(dnp no)
-		(property "Reference" "#PWR096"
+		(property "Reference" "#PWR010"
 			(at 191.6081 92.0264 0)
 			(effects
@@
 			(project "Vendo_main_board"
 				(path "/ce68e045-3b24-4b1f-b4c3-20bce3f1de80/4e895ab7-4f43-4499-a6a7-69405199c565"
-					(reference "#PWR096")
+					(reference "#PWR010")
 					(unit 1)
 				)
@@
 		(dnp no)
 		(fields_autoplaced yes)
-		(property "Reference" "#PWR060"
+		(property "Reference" "#PWR08"
 			(at 172.6493 123.1073 0)
 			(effects
@@
 			(project "Vendo_main_board"
 				(path "/ce68e045-3b24-4b1f-b4c3-20bce3f1de80/4e895ab7-4f43-4499-a6a7-69405199c565"
-					(reference "#PWR060")
+					(reference "#PWR08")
 					(unit 1)
 				)
@@
 		(on_board yes)
 		(dnp no)
-		(property "Reference" "C19"
+		(property "Reference" "C2"
 			(at 97.6817 87.3305 0)
 			(effects
@@
 			(project "Vendo_main_board"
 				(path "/ce68e045-3b24-4b1f-b4c3-20bce3f1de80/4e895ab7-4f43-4499-a6a7-69405199c565"
-					(reference "C19")
+					(reference "C2")
 					(unit 1)
 				)
@@
 		(dnp no)
 		(fields_autoplaced yes)
-		(property "Reference" "R45"
+		(property "Reference" "R2"
 			(at 165.9025 97.5318 0)
 			(effects
@@
 			(project "Vendo_main_board"
 				(path "/ce68e045-3b24-4b1f-b4c3-20bce3f1de80/4e895ab7-4f43-4499-a6a7-69405199c565"
-					(reference "R45")
+					(reference "R2")
 					(unit 1)
 				)
@@
 		(dnp yes)
 		(fields_autoplaced yes)
-		(property "Reference" "C31"
+		(property "Reference" "C5"
 			(at 176.0625 97.5318 0)
 			(effects
@@
 			(project "Vendo_main_board"
 				(path "/ce68e045-3b24-4b1f-b4c3-20bce3f1de80/4e895ab7-4f43-4499-a6a7-69405199c565"
-					(reference "C31")
+					(reference "C5")
 					(unit 1)
 				)
@@
 		(dnp no)
 		(fields_autoplaced yes)
-		(property "Reference" "C20"
+		(property "Reference" "C4"
 			(at 166.9572 111.4763 0)
 			(effects
@@
 			(project "Vendo_main_board"
 				(path "/ce68e045-3b24-4b1f-b4c3-20bce3f1de80/4e895ab7-4f43-4499-a6a7-69405199c565"
-					(reference "C20")
+					(reference "C4")
 					(unit 1)
 				)
@@
 		(dnp no)
 		(fields_autoplaced yes)
-		(property "Reference" "C20"
+		(property "Reference" "C3"
 			(at 132.7029 57.1526 90)
 			(effects
@@
 			(project "Vendo_main_board"
 				(path "/ce68e045-3b24-4b1f-b4c3-20bce3f1de80/4e895ab7-4f43-4499-a6a7-69405199c565"
-					(reference "C20")
+					(reference "C3")
 					(unit 1)
 				)
@@
 		(dnp no)
 		(fields_autoplaced yes)
-		(property "Reference" "R46"
+		(property "Reference" "R3"
 			(at 202.0238 83.7603 0)
 			(effects
@@
 			(project "Vendo_main_board"
 				(path "/ce68e045-3b24-4b1f-b4c3-20bce3f1de80/4e895ab7-4f43-4499-a6a7-69405199c565"
-					(reference "R46")
-					(unit 1)
-				)
+					(reference "R3")
+					(unit 1)
+				)
