File: Vendo_main_board/Vendo_main_board/Vendo_main_board.kicad_sch (KiCad schematic)
At the start: 8 parts, among them J1 Screw_Terminal_01x12, J2 Screw_Terminal_01x12, J3 Screw_Terminal_01x12, J4 Screw_Terminal_01x12

Commit message: -update scheme for modular design
-12V to 5V buck
-5V isolation
-3v3 ldo with wdt
-STM32 blue pill
-dip switch 8 pos with 74HC165
-built in type C programmer
-STLINK 1x4 provisioned
-seven segment port with TM1637 (DIO,CLK)
-relay with 10A & 30A provision , spade connector is put on choosing between 12V supply or external supply , as well on the Common of relay for Ground option
-Coin slot with opto, and loadswitch for it supply 3 pin jst for the port
-slave connector 6 pin jst ,i2c ,5V input for slave seperate gnds
-terminal block for 12V selector for ease of wiring for multiple boards
-terminal io blocks are 16 pin
1button and led with ground pair
12V supply for  device and external supply with grnd pair
relay nc,no and com
esp interrup,sda,scl and gnd for iot connection
Parts:
- removed J1, J2, J3, J4: Screw_Terminal_01x12, TerminalBlock_Phoenix:TerminalBlock_Phoenix_MKDS-1,5-12-5.08_1x12_P5.08mm_Horizontal, symbol Connector:Screw_Terminal_01x12
- added C1, C17, C6: 1uF, Capacitor_SMD:C_0805_2012Metric_Pad1.18x1.45mm_HandSolder, symbol Device:C
- added C10: 3.3nF, Capacitor_SMD:C_0603_1608Metric, symbol Device:C
- added C11: 56pF, Capacitor_SMD:C_0603_1608Metric, symbol Device:C
- added C12, C7: 100uF, Capacitor_SMD:C_1210_3225Metric_Pad1.33x2.70mm_HandSolder, symbol Device:C_Polarized
- added C13, C19: 22uF, Capacitor_SMD:C_1210_3225Metric, symbol Device:C
- added C14, C18, C23, C27, C29, C9: 100nF, Capacitor_SMD:C_0603_1608Metric_Pad1.08x0.95mm_HandSolder, symbol Device:C
- added C15: 10nF, Capacitor_SMD:C_0603_1608Metric_Pad1.08x0.95mm_HandSolder, symbol Device:C
- added C16, C32, C40, C5: 10uF, Capacitor_SMD:C_0805_2012Metric_Pad1.18x1.45mm_HandSolder, symbol Device:C
- added C2, C4: 10uF, Capacitor_SMD:C_1206_3216Metric_Pad1.33x1.80mm_HandSolder, symbol Device:C
- added C20, C24, C28: 10uF, Capacitor_SMD:C_0603_1608Metric_Pad1.08x0.95mm_HandSolder, symbol Device:C
- added C21, C22, C33, C34, C35, C36, C37, C38, C39: 0.1uF, Capacitor_SMD:C_0603_1608Metric, symbol Device:C
- added C25, C26, C30, C31: 20pF, Capacitor_SMD:C_0603_1608Metric, symbol Device:C
- added C3: 470pF, Capacitor_SMD:C_0603_1608Metric_Pad1.08x0.95mm_HandSolder, symbol Device:C
- added C8: 100nF, Capacitor_SMD:C_0603_1608Metric, symbol Device:C
- added D1, D2, D3, D4: LED, LED_SMD:LED_0805_2012Metric_Pad1.15x1.40mm_HandSolder, symbol Device:LED
- added D5: 1N4001, Diode_SMD:D_SOD-123F, symbol pspice:DIODE
- added J1: STLINK, Connector_PinHeader_2.54mm:PinHeader_1x04_P2.54mm_Vertical, symbol Connector:Conn_01x04_Pin
- added J10, J11, J8, J9: Screw_Terminal_01x04, TerminalBlock_MetzConnect:TerminalBlock_MetzConnect_Type055_RT01504HDWU_1x04_P5.00mm_Horizontal, symbol Connector:Screw_Terminal_01x04
- added J12, J13: Screw_Terminal_01x02, TerminalBlock:TerminalBlock_bornier-2_P5.08mm, symbol Connector:Screw_Terminal_01x02
- added J14, J15, J16, J17, J18: 197084013, InnovKits:Spade Conn4.8mm, symbol Vendo_symbol:197084013
- added J2: Conn_01x02_Pin, Connector_PinHeader_2.54mm:PinHeader_1x02_P2.54mm_Vertical, symbol Connector:Conn_01x02_Pin
- added J23: BOOT, Connector_PinSocket_2.54mm:PinSocket_2x03_P2.54mm_Vertical, symbol Connector_Generic:Conn_02x03_Odd_Even
- added J3: Conn_01x08_Pin, Connector_PinHeader_1.00mm:PinHeader_1x08_P1.00mm_Vertical, symbol Connector:Conn_01x08_Pin
- added J4: Conn_01x04_Pin, Connector_PinHeader_2.54mm:PinHeader_1x04_P2.54mm_Vertical, symbol Connector:Conn_01x04_Pin
- added J5: Screw_Terminal_01x03, Connector_JST:JST_EH_B3B-EH-A_1x03_P2.50mm_Vertical, symbol Connector:Conn_01x03_Socket
- added J6, J7: Conn_01x06_Pin, Connector_JST:JST_EH_B6B-EH-A_1x06_P2.50mm_Vertical, symbol Connector:Conn_01x06_Pin
- added JP1, JP4: SolderJumper_3_Open, Jumper:SolderJumper-3_P1.3mm_Open_RoundedPad1.0x1.5mm, symbol Jumper:SolderJumper_3_Open
- added JP2, JP3, JP5: SolderJumper_2_Open, Jumper:SolderJumper-2_P1.3mm_Open_Pad1.0x1.5mm, symbol Jumper:SolderJumper_2_Open
- added JP6, JP7: SolderJumper_2_Open, Jumper:SolderJumper-2_P1.3mm_Open_RoundedPad1.0x1.5mm, symbol Jumper:SolderJumper_2_Open
- added K1: SRD-05VDC-SL-C, Relay_THT:Relay_SPDT_SANYOU_SRD_Series_Form_C, symbol Relay:SANYOU_SRD_Form_C
- added K2: ~, InnovKits:RELAY-TH_SLA-XXVDC-SL-C, symbol Vendo_symbol:SLA-5VDC-SL-C
- added L1: 5.5uH, InnovKits:744325550, symbol pspice:INDUCTOR
- added Q1, Q2: BSS138, Package_TO_SOT_SMD:SOT-23, symbol Transistor_FET:BSS138
- added Q3: S8050, Package_TO_SOT_SMD:SOT-23, symbol Transistor_BJT:Q_NPN_BEC
- added Q4: Q_NMOS_Depletion_GSD, Package_TO_SOT_SMD:SOT-23-3, symbol Device:Q_NMOS_Depletion_GSD
- added Q5: ~, footprints:SOT-23-3_L2.9-W1.6-P1.90-LS2.8-BR, symbol symbol_library:AO3407A
- added R1, R13, R16, R18, R19, R20, R21, R22, R23, R24, R26, R3, R38: 10K, Resistor_SMD:R_0603_1608Metric_Pad0.98x0.95mm_HandSolder, symbol Device:R
- added R10: 10k, Resistor_SMD:R_0603_1608Metric_Pad0.98x0.95mm_HandSolder, symbol Device:R
- added R100, R99: 100k, Resistor_SMD:R_0603_1608Metric, symbol Device:R
- added R11, R12, R29, R30, R37: 1K, Resistor_SMD:R_0603_1608Metric_Pad0.98x0.95mm_HandSolder, symbol Device:R
- added R14, R15: 20, Resistor_SMD:R_0603_1608Metric_Pad0.98x0.95mm_HandSolder, symbol Device:R
- added R17, R27, R28, R34: 4.7k, Resistor_SMD:R_0603_1608Metric_Pad0.98x0.95mm_HandSolder, symbol Device:R
- added R2: 200k, Resistor_SMD:R_0603_1608Metric_Pad0.98x0.95mm_HandSolder, symbol Device:R
- added R25: 1M, Resistor_SMD:R_0603_1608Metric, symbol Device:R
- added R31: 10k, Resistor_SMD:R_0805_2012Metric_Pad1.20x1.40mm_HandSolder, symbol Device:R
- added R32, R33, R35, R41, R42: 1k, Resistor_SMD:R_0805_2012Metric_Pad1.20x1.40mm_HandSolder, symbol Device:R
- added R36: 1k, Resistor_SMD:R_0603_1608Metric_Pad0.98x0.95mm_HandSolder, symbol Device:R
- added R39: 100k, Resistor_SMD:R_0603_1608Metric_Pad0.98x0.95mm_HandSolder, symbol Device:R
- added R4: 40.2K, Resistor_SMD:R_0603_1608Metric_Pad0.98x0.95mm_HandSolder, symbol Device:R
- added R40: 100, Resistor_SMD:R_0603_1608Metric_Pad0.98x0.95mm_HandSolder, symbol Device:R
- added R5: 14k, Resistor_SMD:R_0603_1608Metric_Pad0.98x0.95mm_HandSolder, symbol Device:R
- added R6: 100K, Resistor_SMD:R_0603_1608Metric_Pad0.98x0.95mm_HandSolder, symbol Device:R
- added R7: 147k, Resistor_SMD:R_0603_1608Metric_Pad0.98x0.95mm_HandSolder, symbol Device:R
- added R8: 28k, Resistor_SMD:R_0603_1608Metric_Pad0.98x0.95mm_HandSolder, symbol Device:R
- added R9: 3.3K, Resistor_SMD:R_0805_2012Metric_Pad1.20x1.40mm_HandSolder, symbol Device:R
- added SW1: SW_Push, Button_Switch_SMD:SW_SPST_CK_RS282G05A3, symbol Switch:SW_Push
- added SW2: SW_DIP_x08, Button_Switch_THT:SW_DIP_SPSTx08_Slide_9.78x22.5mm_W7.62mm_P2.54mm, symbol Switch:SW_DIP_x08
- added U1: AP64350SP-13, InnovKits:AP64350SP-13-L, symbol adp650:AP64350SP-13
- added U10: 74HC165, InnovKits:SOIC-16_L9.9-W3.9-P1.27-LS6.0-BL, symbol 74xx:74HC165
- added U11, U12: PC817, InnovKits:APC-817xx-SL_AMB, symbol Isolator:PC817
- added U2: TPS22917DBV, Package_TO_SOT_SMD:SOT-23-6, symbol Power_Management:TPS22917DBV
- added U3: B0505S-2WR3, InnovKits:B_S-2WR2_MNS, symbol 2024-08-29_08-56-51:B0505S-2WR3
- added U4: TPL5010, Package_TO_SOT_SMD:SOT-23-6, symbol Timer:TPL5010
- added U5: TPS73733DCQR, Package_TO_SOT_SMD:SOT-223-6, symbol 2024-09-21_14-21-20:TPS73733DCQR
- added U6: 74AHCT1G125, Package_TO_SOT_SMD:SOT-23-5_HandSoldering, symbol 74xGxx:74AHCT1G125
- added U7: CH340C, Package_SO:SOP-16_4.4x10.4mm_P1.27mm, symbol Interface_USB:CH340C
- added U8: TM1637, InnovKits:SOP-20_L12.8-W7.5-P1.27-LS10.4-BL, symbol Vendo_symbol:TM1637_C2962580
- added U9: STM32F103C8T6, InnovKits:LQFP-48_L7.0-W7.0-P0.50-LS9.0-BL, symbol STM32F103C8T6:STM32F103C8T6
- added USB1: ~, InnovKits:USB-C-SMD_TYPE-C16PIN, symbol TYPEC-allpcb:TYPE-C16PIN
- added Y1: 8MHz, InnovKits:HC-49S_L11.4-W4.9-LS13.4, symbol Device:Crystal
- added Y2: 32.768kHz, InnovKits:OSC-SMD_L3.2-W1.5, symbol Device:Crystal
Connections:
- net +5V: now also C1.2, C12.1, C14.2, C16.2, C24.1, C32.2, C34.2, C9.1, JP1.3 (B), JP2.1 (A), R1.2, R13.1, R16.1, R17.1, R18.1, R19.1, R21.1, R23.1, R24.1, R26.1, R6.1, U10.16 (VCC), U2.1 (VIN), U3.6 (+VO), U4.1 (VDD), U6.5 (VCC), U7.16 (VCC), USB1.A4B9 (VBUS), USB1.B4A9 (VBUS)
- net GNDD: now also C12.2, C14.1, C15.1, C16.1, C17.1, C18.1, C20.1, C21.1, C22.1, C23.2, C24.2, C27.1, C28.1, C29.1, C32.1, C33.1, C34.1, C35.1, C36.1, C37.1, C38.1, C39.1, C6.1, C9.2, J1.4 (Pin_4), J2.2 (Pin_2), J6.6 (Pin_6), J7.6 (Pin_6), J8.2 (Pin_2), J9.4 (Pin_4), R3.1, R37.2, R4.1, R42.1, R9.2, SW1.1, SW2.1, SW2.2, SW2.3, SW2.4, SW2.5, SW2.6, SW2.7, SW2.8, U10.10 (DS), U10.15 (~{CE}), U10.8 (GND), U12.3, U3.4 (0V), U4.2 (GND), U5.3 (GND), U5.6 (TAB), U6.1, U7.1 (GND), U8.1 (GND), U9.23 (VSS), U9.35 (VSS__1), U9.47 (VSS__2), U9.8 (VSSA), USB1.A1B12 (GND), USB1.B1A12 (GND)
- net GNDPWR: now also C10.2, C11.2, C19.2, C2.2, C4.2, C40.2, C5.1, C7.2, D1.1 (K), J10.2 (Pin_2), J10.4 (Pin_4), J12.2 (Pin_2), J13.2 (Pin_2), J18.1_1,1_2, J5.3 (Pin_3), J6.2 (Pin_2), J7.2 (Pin_2), Q3.2 (E), Q4.2 (S), R2.2, R33.1, R38.2, R8.2, U1.7 (GND), U1.EPAD (GND), U12.2, U3.2 (GND)
- new net: C6.2, JP2.2 (B), U2.6 (VOUT), U5.1 (IN), U5.5 (EN)
- new net: JP3.2 (B), R4.2, U4.3 (DELAY/M_RST)
- new net: R16.2, SW2.15, U10.12 (D1)
- new net: C8.2, L1.1, U1.8 (SW)
- new net: R31.2, U11.2
- new net: Q4.1 (G), R38.1, U11.3
- new net: J8.4 (Pin_4), R37.1
- new net: JP6.2 (B), R14.1
- new net: D4.1 (K), D5.1 (K), K1.2, K2.4, Q4.3 (D)
- new net: J5.2 (Pin_2), R32.2, R33.2, R35.1
- new net: C11.1, R5.1, U1.6 (COMP)
- new net: C10.1, R5.2
- new net: C3.2, U2.4 (CT)
- new net: JP1.2 (C), R1.1, U2.3 (ON)
- new net: JP7.2 (B), R15.1
- new net: Q3.3 (C), R39.2, R40.1
- new net: JP4.2 (C), R6.2, U4.6 (~{RST})
- new net: R19.2, SW2.13, U10.14 (D3)
- new net: Q1.1 (G), Q2.2 (S), U7.13 (~{DTR})
- new net: Q1.2 (S), Q2.1 (G), U7.14 (~{RTS})
- new net: D4.2 (A), R36.2
- new net: R35.2, U12.1
- new net: JP5.2 (B), U4.4 (DONE), U6.4
- new net: D2.2 (A), R20.2
- new net: J23.4 (Pin_4), R100.1
- new net: D3.2 (A), R22.2
- new net: C23.1, U7.4 (V3)
- new net: D1.2 (A), R10.2
- new net: R18.2, SW2.14, U10.13 (D2)
- new net: JP3.1 (A), R3.2
- new net: R7.2, R8.1, U1.5 (FB)
- new net: J23.3 (Pin_3), R99.2
- new net: Q3.1 (B), R34.2
- new net: C25.1, C26.1
- new net: R2.1, U1.4 (RT/CLK)
- new net: R21.2, SW2.12, U10.3 (D4)
- new net: Q5.1 (G), R40.2
- new net: R24.2, SW2.10, U10.5 (D6)
- new net: C8.1, U1.1 (BST)
- new net: C15.2, U5.4 (FB)
- new net: R26.2, SW2.9, U10.6 (D7)
- new net: R23.2, SW2.11, U10.4 (D5)
- new net: R13.2, SW2.16, U10.11 (D0)
- new net +3.3V: C17.2, C18.2, C20.2, C27.2, C28.2, C33.2, C35.2, C38.2, C39.2, J1.1 (Pin_1), J23.1 (Pin_1), J23.2 (Pin_2), R11.1, R12.1, R20.1, R22.1, R27.1, R28.1, R29.1, R30.1, R41.1, R9.1, U11.1, U5.2 (OUT), U8.16 (VDD), U9.24 (VDD), U9.36 (VDD__1), U9.48 (VDD__2), U9.9 (VDDA)
- new net +5VA: C13.1, C19.1, C5.2, C7.1, D5.2 (A), J6.1 (Pin_1), J7.1 (Pin_1), K1.5, K2.3, L1.2, R10.1, R32.1, R36.1, R7.1, U11.4, U3.1 (VIN)
- new net 12V: C2.1, C4.1, C40.1, J10.1 (Pin_1), J14.1_1,1_2, Q5.2 (S), R39.1, U1.2 (VIN), U1.3 (EN)
- new net 12VA: J5.1 (Pin_1), Q5.3 (D)
- new net 12V_SEL: J11.1 (Pin_1), J11.3 (Pin_3), J12.1 (Pin_1), J13.1 (Pin_1), J15.1_1,1_2, K1.3, K1.4, K2.1, K2.2
- new net 3V3_EN: JP1.1 (A), JP4.1 (A)
- new net BUTTON_1: C36.2, J8.1 (Pin_1), R29.2
- new net COM: J11.2 (Pin_2), J16.1_1,1_2, K1.1, K2.5, K2.6
- new net CTRL_DCI1: U9.46 (PB9)
- new net D+: JP7.1 (A), U7.5 (UD+), USB1.A6 (DP1), USB1.B6 (DP2)
- new net D-: JP6.1 (A), U7.6 (UD-), USB1.A7 (DN1), USB1.B7 (DN2)
- new net DC_DRV_1: R31.1, U9.16 (PA6)
- new net EN_COIN: R34.1, U9.14 (PA4)
- new net ESP_INT: C37.2, J9.1 (Pin_1), R30.2, U9.41 (PB5)
- new net EXT: J10.3 (Pin_3), J17.1_1,1_2
- new net GND: C1.1, C13.2, C3.1, C30.1, C31.1, J23.5 (Pin_5), J23.6 (Pin_6), U2.2 (GND), U6.3 (GND)
- new net GRID1: J4.1 (Pin_1), U8.15 (GRID1)
- new net GRID2: J4.2 (Pin_2), U8.14 (GRID2)
- new net GRID3: J4.3 (Pin_3), U8.13 (GRID3)
- new net GRID4: J4.4 (Pin_4), U8.12 (GRID4)
- new net I2C_CONF: J2.1 (Pin_1), R11.2, U9.29 (PA8)
- new net LED_P: J8.3 (Pin_3), U9.40 (PB4)
- new net OSCIN: C25.2, R25.1, U9.5 (PD0_OSC_IN), Y1.2
- new net OSCOUT: C26.2, R25.2, U9.6 (PD1_OSC_OUT), Y1.1
- new net PA11: R14.2, U9.32 (PA11)
- new net PA12: R15.2, R17.2, U9.33 (PA12)
- new net PC14: C30.2, U9.3 (PC14-OSC32_IN), Y2.2
- new net PC15: C31.2, U9.4 (PC15-OSC32_OUT), Y2.1
- new net SEG1/KS1: J3.1 (Pin_1), U8.2 (SEG1/KS1)
- new net SEG2/KS2: J3.2 (Pin_2), U8.3 (SEG2/KS2)
- new net SEG3/KS3: J3.3 (Pin_3), U8.4 (SEG3/KS3)
- new net SEG4/KS4: J3.4 (Pin_4), U8.5 (SEG4/KS4)
- new net SEG5/KS5: J3.5 (Pin_5), U8.6 (SEG5/KS5)
- new net SEG6/KS6: J3.6 (Pin_6), U8.7 (SEG6/KS6)
- new net SEG7/KS7: J3.7 (Pin_7), U8.8 (SEG7/KS7)
- new net SEG8/KS8: J3.8 (Pin_8), U8.9 (SEG8/KS8)
- new net SEG_CLK: R27.2, U8.18 (CLK), U9.21 (PB10)
- new net SEG_DIO: R28.2, U8.17 (DIO), U9.22 (PB11)
- new net STM32_BOOT0: Q2.3 (D), R100.2, U9.44 (BOOT0)
- new net STM32_BOOT1: R99.1, U9.20 (PB2)
- new net STM32_IN1: R41.2, R42.2, U12.4, U9.15 (PA5)
- new net STM32_RX: D2.1 (K), U7.2 (TXD), U9.31 (PA10)
- new net STM32_SCL: J6.5 (Pin_5), J7.5 (Pin_5), J9.2 (Pin_2), U9.42 (PB6)
- new net STM32_SDA: J6.4 (Pin_4), J7.4 (Pin_4), J9.3 (Pin_3), U9.43 (PB7)
- new net STM32_SWCLK: J1.3 (Pin_3), U9.37 (PA14)
- new net STM32_SWDIO: J1.2 (Pin_2), U9.34 (PA13)
- new net STM32_TX: D3.1 (K), U7.3 (RXD), U9.30 (PA9)
- new net STM_RST: C21.2, C22.2, C29.2, JP4.3 (B), Q1.3 (D), R12.2, SW1.2, U9.7 (NRST)
- new net TMR_CLK: U10.2 (CP), U9.26 (PB13)
- new net TMR_DATA: U10.9 (Q7), U9.28 (PB15)
- new net TMR_LOAD: U10.1 (~{PL}), U9.27 (PB14)
- new net UART_RX1: U9.13 (PA3)
- new net UART_TX1: U9.12 (PA2)
- new net VBAT: U9.1 (VBAT)
- new net WDT_DONE: JP5.1 (A), U6.2, U9.17 (PA7)
- no-connect marks 6 -> 29
Other:
- removed sheet 3V3_LDO_WITH_WDT
- removed sheet 8_CHANNEL_RELAY
- removed sheet COIN_SLOT_ISO
- removed sheet ESP32_MAIN_MCU
- removed sheet IO_EXPANDER
- removed sheet NON_ISO_5V_BUCK
- removed sheet USB_TYPE_C_PROGRAMMER
- removed sheet VOLTAGE_ISOLATOR
- note added: "3V3 REGULATOR"
- note added: "COIN SLOT"
- note added: "CONNECTOR-FOR-SLAVE"
- note added: "D"
- note added: "FC4SDCBMF8"
- note added: "G"
- note added: "IF THE PCB IS MASTER POPULATE THIS"
- note added: "ISOLATED POWER"
- note added: "Output Capacity 5V, 400mA"
- note added: "PROGRAMMER"
- note added: "RELAY"
- note added: "RELAY1"
- note added: "S"
- note added: "SEVEN_SEGMENT PORT"
- note added: "STM32 BLUEPILL"
- note added: "STM32 CRYSTAL"
- note added: "Songle Relay SLA-5VDC-SL-C"
- note added: "TERMINAL BLOCK IO/s"
- note added: "TIMER CONFIGURATION"
- note added: "WATCHDOG TIMER"
- note added: "https://stm32-base.org/boards/STM32F103C8T6-Blue-Pill.html"
- note removed: "16 BIT IO EXPANDER"
- note removed: "3V3 LDO WITH WDT"
- note removed: "5V NON ISO BUCK"
- note removed: "8_CHANNEL_RELAY"
- note removed: "COIN SLOT IO"
- note removed: "ESP32 MCU"
- note removed: "OUTPUT TERMINAL BLOCK"
- note removed: "POWER ISOLATOR"
- note removed: "TYPE C PROG"
- moved on the sheet: H1, H2, H3, H4

Commit message: -scheme edit and update
Edits
-Add 1x04(2.54mm pitch_)for programmer FTDI,STLINK and USB
- coin slot terminal block footprint
-jumper for optoclouper option for DNP
-loadswitch for coin clot have jumper for DNP purposes
-100k interrup value added
-MCU reset on WDT,WDT on 3.3V
-AMS117 added for 3.3V
-provision for isolator jumper
-update LCSC
-update BOM pricing
Removed
- type c programer
- buffer on wdt
- ldo 3.3v replaced by ams117 3.3
PS:
-Terminal block not yet change might be some changes waiting for go signal
-DIP switch no LCSC might be on shopee
Parts:
- removed C14, C23, C29: 100nF, Capacitor_SMD:C_0603_1608Metric_Pad1.08x0.95mm_HandSolder, symbol Device:C
- removed C15: 10nF, Capacitor_SMD:C_0603_1608Metric_Pad1.08x0.95mm_HandSolder, symbol Device:C
- removed C24: 10uF, Capacitor_SMD:C_0603_1608Metric_Pad1.08x0.95mm_HandSolder, symbol Device:C
- removed D3: LED, LED_SMD:LED_0805_2012Metric_Pad1.15x1.40mm_HandSolder, symbol Device:LED
- removed JP1, JP4: SolderJumper_3_Open, Jumper:SolderJumper-3_P1.3mm_Open_RoundedPad1.0x1.5mm, symbol Jumper:SolderJumper_3_Open
- removed Q1, Q2: BSS138, Package_TO_SOT_SMD:SOT-23, symbol Transistor_FET:BSS138
- removed R20, R22: 10K, Resistor_SMD:R_0603_1608Metric_Pad0.98x0.95mm_HandSolder, symbol Device:R
- removed U2: TPS22917DBV, Package_TO_SOT_SMD:SOT-23-6, symbol Power_Management:TPS22917DBV
- removed U5: TPS73733DCQR, Package_TO_SOT_SMD:SOT-223-6, symbol 2024-09-21_14-21-20:TPS73733DCQR
- removed U6: 74AHCT1G125, Package_TO_SOT_SMD:SOT-23-5_HandSoldering, symbol 74xGxx:74AHCT1G125
- removed U7: CH340C, Package_SO:SOP-16_4.4x10.4mm_P1.27mm, symbol Interface_USB:CH340C
- removed USB1: ~, InnovKits:USB-C-SMD_TYPE-C16PIN, symbol TYPEC-allpcb:TYPE-C16PIN
- added J19: FTDI, Connector_PinHeader_2.54mm:PinHeader_1x04_P2.54mm_Vertical, symbol Connector:Conn_01x04_Pin
- added J20: USB, Connector_PinHeader_2.54mm:PinHeader_1x04_P2.54mm_Vertical, symbol Connector:Conn_01x04_Pin
- added JP1, JP4: SolderJumper_2_Open, Jumper:SolderJumper-2_P1.3mm_Open_RoundedPad1.0x1.5mm, symbol Jumper:SolderJumper_2_Open
- added U2: AMS1117-3.3, Package_TO_SOT_SMD:SOT-223-3_TabPin2, symbol Regulator_Linear:AMS1117-3.3
- C1: value 1uF -> 22uF; footprint Capacitor_SMD:C_0805_2012Metric_Pad1.18x1.45mm_HandSolder -> Capacitor_SMD:C_0603_1608Metric; LCSC C49678 -> C59461; Price (none) -> 0.0101
- C10: Price (none) -> 0.0028
- C12, C7: Price (none) -> 0.5192
- C13, C19: Price (none) -> 0.1478
- C16, C32, C40, C5: LCSC C15850 -> C84416; Price (none) -> 0.0288
- C17, C6: Price (none) -> 0.0053
- C18, C27, C9: Price (none) -> 0.0031
- C2, C4: Price (none) -> 0.0973
- C20, C28: LCSC C19702 -> C85713; Price (none) -> 0.0106
- C21, C22, C34, C36, C37: value 0.1uF -> 100nF; footprint Capacitor_SMD:C_0603_1608Metric -> Capacitor_SMD:C_0603_1608Metric_Pad1.08x0.95mm_HandSolder; LCSC C80516 -> C14663; Price (none) -> 0.0031
- C25, C26, C30, C31: LCSC (none) -> C1648; Price (none) -> 0.0059
- C3: value 470pF -> 22uF; footprint Capacitor_SMD:C_0603_1608Metric_Pad1.08x0.95mm_HandSolder -> Capacitor_SMD:C_0603_1608Metric; LCSC C106211 -> C59461; Price (none) -> 0.0101
- C33, C35, C38, C39: value 0.1uF -> 100nF; footprint Capacitor_SMD:C_0603_1608Metric -> Capacitor_SMD:C_0603_1608Metric_Pad1.08x0.95mm_HandSolder; LCSC (none) -> C14663; Price (none) -> 0.0031
- C8: footprint Capacitor_SMD:C_0603_1608Metric -> Capacitor_SMD:C_0603_1608Metric_Pad1.08x0.95mm_HandSolder; LCSC WITH STOCK -> C14663; Price (none) -> 0.0031
- D1, D2, D4: Price (none) -> 0.0163
- D5: Price (none) -> 0.0076
- J5: footprint Connector_JST:JST_EH_B3B-EH-A_1x03_P2.50mm_Vertical -> TerminalBlock:TerminalBlock_bornier-3_P5.08mm
- JP2, JP5: footprint Jumper:SolderJumper-2_P1.3mm_Open_Pad1.0x1.5mm -> Jumper:SolderJumper-2_P1.3mm_Open_RoundedPad1.0x1.5mm; now in the parts list
- JP3: footprint Jumper:SolderJumper-2_P1.3mm_Open_Pad1.0x1.5mm -> Jumper:SolderJumper-2_P1.3mm_Open_RoundedPad1.0x1.5mm
- K1: Price (none) -> 0.4863
- K2: LSCC (none) -> C688870; Price (none) -> 1.2933
- L1: Price (none) -> 1.4510
- Q3: Price (none) -> 0.0061
- Q4: Price (none) -> 0.0352
- R1: value 10K -> 1k; LCSC C99782 -> C21190; Price (none) -> 0.0016; now fitted
- R10: value 10k -> 10K; footprint Resistor_SMD:R_0603_1608Metric_Pad0.98x0.95mm_HandSolder -> Resistor_SMD:R_0805_2012Metric_Pad1.20x1.40mm_HandSolder; LCSC WITH STOCK -> C2930231; Price (none) -> 0.0017
- R100, R99: footprint Resistor_SMD:R_0603_1608Metric -> Resistor_SMD:R_0603_1608Metric_Pad0.98x0.95mm_HandSolder; LCSC (none) -> C14675; Price (none) -> 0.0014
- R11, R12, R29, R37: value 1K -> 1k; Price (none) -> 0.0016
- R13, R16, R18, R19, R21, R23, R24, R26: footprint Resistor_SMD:R_0603_1608Metric_Pad0.98x0.95mm_HandSolder -> Resistor_SMD:R_0805_2012Metric_Pad1.20x1.40mm_HandSolder; LCSC C21190 -> C2930231; Price (none) -> 0.0017
- R14, R15: now not fitted
- R17: LCSC C21190 -> C99782; Price (none) -> 0.20810; now not fitted
- R2, R36: Price (none) -> 0.0016
- R25: LCSC (none) -> C105578; Price (none) -> 0.0016
- R27, R28: LCSC C21190 -> C99782; Price (none) -> 0.20810
- R3, R38: footprint Resistor_SMD:R_0603_1608Metric_Pad0.98x0.95mm_HandSolder -> Resistor_SMD:R_0805_2012Metric_Pad1.20x1.40mm_HandSolder; LCSC C25804 -> C2930231; Price (none) -> 0.0017
- R30: value 1K -> 100K; LCSC C21190 -> C105574; Price (none) -> 0.0016
- R31: value 10k -> 10K; LCSC C137786 -> C2930231; Price (none) -> 0.0017
- R32, R33, R35, R41, R42: footprint Resistor_SMD:R_0805_2012Metric_Pad1.20x1.40mm_HandSolder -> Resistor_SMD:R_0603_1608Metric_Pad0.98x0.95mm_HandSolder; Price (none) -> 0.0016
- R39: Price 0.20810 -> 0.0014
- R4: Price (none) -> 0.0015
- R40: Price 0.20810 -> 0.0059
- R5, R7, R8: Price (none) -> 0.0012
- R6: LCSC C21190 -> C105574; Price (none) -> 0.0016
- R9: LCSC C21190 -> C2907249; Price (none) -> 0.0020
- SW1: Price (none) -> 0.3508
- U1: Price (none) -> 0.9176
- U10: Price (none) -> 0.212
- U11, U12: Price (none) -> 0.0969
- U3: Price (none) -> 1.2352
- U4: Price (none) -> 0.3523
- U8: LCSC (none) -> C5337160; Price (none) -> 0.2428
- U9: LCSC (none) -> C8734; Price (none) -> 1.3968
- Y1: Price (none) -> 0.2934
- Y2: Price (none) -> 0.1842
Connections:
- net +3.3V: now also C3.2, C9.1, JP2.1 (A), R6.1, U4.1 (VDD), U2.2 (VO)
- net +5V: now also C6.2, J19.1 (Pin_1), J20.1 (Pin_1), JP1.2 (B), U2.3 (VI); no longer C9.1, JP2.1 (A), R1.2, R6.1, U4.1 (VDD)
- net +5VA: now also JP1.1 (A)
- net 12V: now also JP5.1 (A)
- net 12VA: now also JP5.2 (B)
- net BUTTON_1: now also U9.39 (PB3)
- net D+: now also J20.3 (Pin_3)
- net D-: now also J20.2 (Pin_2)
- net GND: now also R1.2; no longer C1.1, C3.1
- net GNDD: now also C1.1, C3.1, J19.4 (Pin_4), J20.4 (Pin_4), U2.1 (GND)
- net STM32_IN1: now also JP4.2 (B)
- net STM32_RX: now also J19.3 (Pin_3); no longer D2.1 (K)
- net STM32_TX: now also J19.2 (Pin_2)
- net STM_RST: now also R6.2, U4.6 (~{RST})
- net WDT_DONE: now also U4.4 (DONE); no longer JP5.1 (A)
- net at JP2.2 (B): now also D2.2 (A); no longer C6.2
- net at J5.2 (Pin_2), R32.2, R33.2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: now also JP4.1 (A)
- net at R1.1: now also D2.1 (K)
- no-connect marks 29 -> 15
Other:
- moved on the sheet: C17, C18, C20, C6, J1, J2, R11, R9

Commit message: -scheme edit
-update lscs inductor and cap of iso
-update footprint inductor
-move esp_int on the jst pin
-isolate the supply for the seven segment other boards
-add 1x04 jst/ header for seven segment dio.clk and 3v3 supply
Parts:
- added J21: Conn_01x04_Pin, Connector_PinHeader_2.54mm:PinHeader_1x04_P2.54mm_Vertical, symbol Connector:Conn_01x04_Pin
- added TP1: TestPoint, symbol Connector:TestPoint
- C12, C7: LCSC C394395 -> C883598
- L1: value 5.5uH -> 6.8uH; footprint InnovKits:744325550 -> InnovKits:IND-SMD_L11.5-W10.0_FXL1040; LCSC C2761919 -> C167231; Price 1.4510 -> 0.3926
Connections:
- net +3.3V: now also J21.1 (Pin_1); no longer C27.2, C28.2, R27.1, R28.1, U8.16 (VDD)
- net ESP_INT: now also J6.3 (Pin_3), J7.3 (Pin_3)
- net GNDD: no longer C27.1, C28.1, U8.1 (GND)
- net SEG_CLK: now also J21.2 (Pin_2); no longer R27.2, U8.18 (CLK)
- net SEG_DIO: now also J21.3 (Pin_3); no longer R28.2, U8.17 (DIO)
- net at JP3.2 (B), R4.2, U4.3 (DELAY/M_RST): now also TP1.1
- new net +3.3VA: C27.2, C28.2, R27.1, R28.1, U8.16 (VDD)
- new net CLK: R27.2, U8.18 (CLK)
- new net DIO: R28.2, U8.17 (DIO)
- new net GND1: C27.1, C28.1, J21.4 (Pin_4), U8.1 (GND)
- no-connect marks 15 -> 13
Other:
- note added: "SEVEN_SEGMENT PORT(ANOTHER BOARD)"
- note removed: "SEVEN_SEGMENT PORT"

Commit message: -pcb , update scheme tweak
-pcb placement
-remove USB prog related , no need we have ftdi stlink
Parts:
- removed C27: 100nF, Capacitor_SMD:C_0603_1608Metric_Pad1.08x0.95mm_HandSolder, symbol Device:C
- removed C28: 10uF, Capacitor_SMD:C_0603_1608Metric_Pad1.08x0.95mm_HandSolder, symbol Device:C
- removed J20: USB, Connector_PinHeader_2.54mm:PinHeader_1x04_P2.54mm_Vertical, symbol Connector:Conn_01x04_Pin
- removed J3: Conn_01x08_Pin, Connector_PinHeader_1.00mm:PinHeader_1x08_P1.00mm_Vertical, symbol Connector:Conn_01x08_Pin
- removed J4: Conn_01x04_Pin, Connector_PinHeader_2.54mm:PinHeader_1x04_P2.54mm_Vertical, symbol Connector:Conn_01x04_Pin
- removed JP2, JP6, JP7: SolderJumper_2_Open, Jumper:SolderJumper-2_P1.3mm_Open_RoundedPad1.0x1.5mm, symbol Jumper:SolderJumper_2_Open
- removed R100, R99: 100k, Resistor_SMD:R_0603_1608Metric_Pad0.98x0.95mm_HandSolder, symbol Device:R
- removed R17, R27, R28: 4.7k, Resistor_SMD:R_0603_1608Metric_Pad0.98x0.95mm_HandSolder, symbol Device:R
- removed U8: TM1637, InnovKits:SOP-20_L12.8-W7.5-P1.27-LS10.4-BL, symbol Vendo_symbol:TM1637_C2962580
- added TP2: TestPoint, TestPoint:TestPoint_Pad_D1.0mm, symbol Connector:TestPoint
- J12, J13: footprint TerminalBlock:TerminalBlock_bornier-2_P5.08mm -> TerminalBlock_MetzConnect:TerminalBlock_MetzConnect_Type073_RT02602HBLU_1x02_P5.08mm_Horizontal
- J5: footprint TerminalBlock:TerminalBlock_bornier-3_P5.08mm -> TerminalBlock_MetzConnect:TerminalBlock_MetzConnect_Type073_RT02603HBLU_1x03_P5.08mm_Horizontal
- R14, R15: value 20 -> 100k; LCSC C21190 -> C14675; Price (none) -> 0.0014; now fitted
- R3: footprint Resistor_SMD:R_0805_2012Metric_Pad1.20x1.40mm_HandSolder -> Resistor_SMD:R_0603_1608Metric_Pad0.98x0.95mm_HandSolder
- TP1: footprint (none) -> TestPoint:TestPoint_Pad_D1.0mm
Connections:
- net +3.3V: now also D2.2 (A)
- net +5VA: now also J6.6 (Pin_6); no longer J6.1 (Pin_1)
- net 12V_SEL: now also J12.2 (Pin_2); no longer J12.1 (Pin_1)
- net ESP_INT: now also J6.4 (Pin_4); no longer J6.3 (Pin_3)
- net GNDD: now also J6.1 (Pin_1); no longer J6.6 (Pin_6)
- net GNDPWR: now also J12.1 (Pin_1), J6.5 (Pin_5); no longer J12.2 (Pin_2), J6.2 (Pin_2)
- net PA11: no longer R14.2
- net PA12: no longer R15.2
- net STM32_BOOT0: now also R15.2
- net STM32_BOOT1: now also R14.1
- net STM32_SCL: now also J6.2 (Pin_2); no longer J6.5 (Pin_5)
- net STM32_SDA: now also J6.3 (Pin_3); no longer J6.4 (Pin_4)
- net STM_RST: now also TP2.1
- net at R15.1: now also J23.4 (Pin_4)
- net at J23.3 (Pin_3): now also R14.2
- no-connect marks 13 -> 9
Other:
- note removed: "SEVEN_SEGMENT PORT(ANOTHER BOARD)"
