File: Vendo_main_board/Vendo_main_board/Vendo_main_board.kicad_sch (KiCad schematic)
At the start: 121 parts, among them J1 STLINK, J10 Screw_Terminal_01x04, J11 Screw_Terminal_01x04, J12 Screw_Terminal_01x02, J13 Screw_Terminal_01x02, J14 197084013, J15 197084013, J16 197084013, J17 197084013, J18 197084013, J19 FTDI, J2 Conn_01x02_Pin, J21 Conn_01x04_Pin, J23 BOOT, J5 Screw_Terminal_01x03, J6 Conn_01x06_Pin, J7 Conn_01x06_Pin, J8 Screw_Terminal_01x04, J9 Screw_Terminal_01x04, K1 SRD-05VDC-SL-C, Q3 S8050, Q4 Q_NMOS_Depletion_GSD, SW1 SW_Push, SW2 SW_DIP_x08, U1 AP64350SP-13, U10 74HC165, U11 PC817, U12 PC817, U2 AMS1117-3.3, U3 B0505S-2WR3, U4 TPL5010, U9 STM32F103C8T6, Y1 8MHz, Y2 32.768kHz

Commit message: -scheme update by charles
1. Used standard input and output nodes
2. Fixed GND connection of BOOT0 and BOOT1 (initially connected to Analog GND)
3. Removed redundant 100K pull up WDT RST Pin
4. Removed Nets on unconnected STM Pins
5. Fixed GND of Oscillator
6. Added 5V and 12V option to LED, removed LED as direct LED Drive
7. Renamed ESP INT to I2C INT
8. Changed 12V to 12VA, removed nets, used power rail symbol instead
9. Simplified 12V Logic
10. removed WDT, STM has internal WDT
11. Added DPDT Config to Relay Logic
12. Added Pullup I2C Line
13. Fixed 5V logic with 3.3V V Logic on 7Seg Driver
14. Added Auxiliary Pins
15.Added Debug LEDs,
Updated Footprints
Parts:
- removed C1: 22uF, Capacitor_SMD:C_0603_1608Metric, symbol Device:C
- removed C12, C7: 100uF, Capacitor_SMD:C_1210_3225Metric_Pad1.33x2.70mm_HandSolder, symbol Device:C_Polarized
- removed C17: 1uF, Capacitor_SMD:C_0805_2012Metric_Pad1.18x1.45mm_HandSolder, symbol Device:C
- removed C18, C22, C34, C36: 100nF, Capacitor_SMD:C_0603_1608Metric_Pad1.08x0.95mm_HandSolder, symbol Device:C
- removed C20: 10uF, Capacitor_SMD:C_0603_1608Metric_Pad1.08x0.95mm_HandSolder, symbol Device:C
- removed C32, C40: 10uF, Capacitor_SMD:C_0805_2012Metric_Pad1.18x1.45mm_HandSolder, symbol Device:C
- removed D1, D2: LED, LED_SMD:LED_0805_2012Metric_Pad1.15x1.40mm_HandSolder, symbol Device:LED
- removed J1: STLINK, Connector_PinHeader_2.54mm:PinHeader_1x04_P2.54mm_Vertical, symbol Connector:Conn_01x04_Pin
- removed J10, J11, J8, J9: Screw_Terminal_01x04, TerminalBlock_MetzConnect:TerminalBlock_MetzConnect_Type055_RT01504HDWU_1x04_P5.00mm_Horizontal, symbol Connector:Screw_Terminal_01x04
- removed J12, J13: Screw_Terminal_01x02, TerminalBlock_MetzConnect:TerminalBlock_MetzConnect_Type073_RT02602HBLU_1x02_P5.08mm_Horizontal, symbol Connector:Screw_Terminal_01x02
- removed J14, J15, J16, J17, J18: 197084013, InnovKits:Spade Conn4.8mm, symbol Vendo_symbol:197084013
- removed J19: FTDI, Connector_PinHeader_2.54mm:PinHeader_1x04_P2.54mm_Vertical, symbol Connector:Conn_01x04_Pin
- removed J2: Conn_01x02_Pin, Connector_PinHeader_2.54mm:PinHeader_1x02_P2.54mm_Vertical, symbol Connector:Conn_01x02_Pin
- removed J21: Conn_01x04_Pin, Connector_PinHeader_2.54mm:PinHeader_1x04_P2.54mm_Vertical, symbol Connector:Conn_01x04_Pin
- removed J5: Screw_Terminal_01x03, TerminalBlock_MetzConnect:TerminalBlock_MetzConnect_Type073_RT02603HBLU_1x03_P5.08mm_Horizontal, symbol Connector:Conn_01x03_Socket
- removed J6, J7: Conn_01x06_Pin, Connector_JST:JST_EH_B6B-EH-A_1x06_P2.50mm_Vertical, symbol Connector:Conn_01x06_Pin
- removed K1: SRD-05VDC-SL-C, Relay_THT:Relay_SPDT_SANYOU_SRD_Series_Form_C, symbol Relay:SANYOU_SRD_Form_C
- removed Q3: S8050, Package_TO_SOT_SMD:SOT-23, symbol Transistor_BJT:Q_NPN_BEC
- removed Q5: ~, footprints:SOT-23-3_L2.9-W1.6-P1.90-LS2.8-BR, symbol symbol_library:AO3407A
- removed R1, R37: 1k, Resistor_SMD:R_0603_1608Metric_Pad0.98x0.95mm_HandSolder, symbol Device:R
- removed R10, R19, R23, R24, R26, R31: 10K, Resistor_SMD:R_0805_2012Metric_Pad1.20x1.40mm_HandSolder, symbol Device:R
- removed R15, R39: 100k, Resistor_SMD:R_0603_1608Metric_Pad0.98x0.95mm_HandSolder, symbol Device:R
- removed R34: 4.7k, Resistor_SMD:R_0603_1608Metric_Pad0.98x0.95mm_HandSolder, symbol Device:R
- removed R4: 40.2K, Resistor_SMD:R_0603_1608Metric_Pad0.98x0.95mm_HandSolder, symbol Device:R
- removed R40: 100, Resistor_SMD:R_0603_1608Metric_Pad0.98x0.95mm_HandSolder, symbol Device:R
- removed R6: 100K, Resistor_SMD:R_0603_1608Metric_Pad0.98x0.95mm_HandSolder, symbol Device:R
- removed SW2: SW_DIP_x08, Button_Switch_THT:SW_DIP_SPSTx08_Slide_9.78x22.5mm_W7.62mm_P2.54mm, symbol Switch:SW_DIP_x08
- removed TP1, TP2: TestPoint, TestPoint:TestPoint_Pad_D1.0mm, symbol Connector:TestPoint
- removed U10: 74HC165, InnovKits:SOIC-16_L9.9-W3.9-P1.27-LS6.0-BL, symbol 74xx:74HC165
- removed U11: PC817, InnovKits:APC-817xx-SL_AMB, symbol Isolator:PC817
- removed U2: AMS1117-3.3, Package_TO_SOT_SMD:SOT-223-3_TabPin2, symbol Regulator_Linear:AMS1117-3.3
- removed U3: B0505S-2WR3, InnovKits:B_S-2WR2_MNS, symbol 2024-08-29_08-56-51:B0505S-2WR3
- removed U4: TPL5010, Package_TO_SOT_SMD:SOT-23-6, symbol Timer:TPL5010
- added C2: 1uF, Capacitor_SMD:C_0805_2012Metric_Pad1.18x1.45mm_HandSolder, symbol Device:C
- added C8: 100nF, Capacitor_SMD:C_0603_1608Metric_Pad1.08x0.95mm_HandSolder, symbol Device:C
- added D4, D6, D7: LED, LED_SMD:LED_0805_2012Metric_Pad1.15x1.40mm_HandSolder, symbol Device:LED
- added J1, J6: Screw_Terminal_01x04, TerminalBlock:TerminalBlock_Xinya_XY308-2.54-4P_1x04_P2.54mm_Horizontal, symbol Connector:Screw_Terminal_01x04
- added J10: Screw_Terminal_01x03, TerminalBlock:TerminalBlock_Xinya_XY308-2.54-3P_1x03_P2.54mm_Horizontal, symbol Connector:Screw_Terminal_01x03
- added J11: Screw_Terminal_01x02, TerminalBlock_MetzConnect:TerminalBlock_MetzConnect_Type073_RT02602HBLU_1x02_P5.08mm_Horizontal, symbol Connector:Screw_Terminal_01x02
- added J12: Screw_Terminal_01x03, TerminalBlock_MetzConnect:TerminalBlock_MetzConnect_Type073_RT02603HBLU_1x03_P5.08mm_Horizontal, symbol Connector:Screw_Terminal_01x03
- added J2: Barrel_Jack_MountingPin, Connector_BarrelJack:BarrelJack_GCT_DCJ200-10-A_Horizontal, symbol Connector:Barrel_Jack_MountingPin
- added J3, J4: Conn_01x05_Pin, Connector_JST:JST_EH_B5B-EH-A_1x05_P2.50mm_Vertical, symbol Connector:Conn_01x05_Pin
- added J7: FTDI, Connector_PinHeader_2.54mm:PinHeader_1x04_P2.54mm_Vertical, symbol Connector:Conn_01x04_Pin
- added J9: Conn_01x04_Pin, Connector_JST:JST_EH_B4B-EH-A_1x04_P2.50mm_Vertical, symbol Connector:Conn_01x04_Pin
- added JP10, JP7: Jumper_3_Open, Connector_PinHeader_2.54mm:PinHeader_1x03_P2.54mm_Vertical, symbol Jumper:Jumper_3_Open
- added JP2: SolderJumper_2_Open, Jumper:SolderJumper-2_P1.3mm_Open_RoundedPad1.0x1.5mm, symbol Jumper:SolderJumper_2_Open
- added JP4: SolderJumper_2_Open, Connector_PinHeader_2.54mm:PinHeader_1x02_P2.54mm_Vertical, symbol Jumper:SolderJumper_2_Open
- added JP6, JP9: SolderJumper_3_Open, Jumper:SolderJumper-3_P1.3mm_Open_Pad1.0x1.5mm_NumberLabels, symbol Jumper:SolderJumper_3_Open
- added Q1, Q3: Q_NMOS_Depletion_GSD, Package_TO_SOT_SMD:SOT-23-3, symbol Device:Q_NMOS_Depletion_GSD
- added R17: 100K, Resistor_SMD:R_0603_1608Metric_Pad0.98x0.95mm_HandSolder, symbol Device:R
- added R2: 4.7K, Resistor_SMD:R_0603_1608Metric_Pad0.98x0.95mm_HandSolder, symbol Device:R
- added R27, R29, R30: 1K, Resistor_SMD:R_0603_1608Metric_Pad0.98x0.95mm_HandSolder, symbol Device:R
- added SW2, SW3, SW4: SW_Push, Button_Switch_THT:SW_PUSH_6mm_H5mm, symbol Switch:SW_Push
- added SW5: SW_Slide_DPDT, InnovKits:DPDT_PUSH, symbol Switch:SW_Slide_DPDT
- added U1: AMS1117-3.3, Package_TO_SOT_SMD:SOT-223-3_TabPin2, symbol Regulator_Linear:AMS1117-3.3
- C16: value 10uF -> 100nF; footprint Capacitor_SMD:C_0805_2012Metric_Pad1.18x1.45mm_HandSolder -> Capacitor_SMD:C_0603_1608Metric_Pad1.08x0.95mm_HandSolder; LCSC C84416 -> C14663; Price 0.0288 -> 0.0031
- C17: renamed from C21; value 100nF -> 1uF
- C5: value 10uF -> 22uF; footprint Capacitor_SMD:C_0805_2012Metric_Pad1.18x1.45mm_HandSolder -> Capacitor_SMD:C_0603_1608Metric; LCSC C84416 -> C59461; Price 0.0288 -> 0.0101
- C9: value 100nF -> 10uF; LCSC C14663 -> C85713; Price 0.0031 -> 0.0106
- H1, H2, H3, H4: footprint MountingHole:MountingHole_3.2mm_M3 -> MountingHole:MountingHole_3.2mm_M3_DIN965_Pad_TopBottom
- JP3, JP5: footprint Jumper:SolderJumper-2_P1.3mm_Open_RoundedPad1.0x1.5mm -> Connector_PinHeader_2.54mm:PinHeader_1x02_P2.54mm_Vertical
- R10: renamed from R29; value 1k -> 1K
- R11: value 1k -> 10K; footprint Resistor_SMD:R_0603_1608Metric_Pad0.98x0.95mm_HandSolder -> Resistor_SMD:R_0805_2012Metric_Pad1.20x1.40mm_HandSolder; LCSC C21190 -> C2930231; Price 0.0016 -> 0.0017
- R12: value 1k -> 10K
- R13, R16, R18: footprint Resistor_SMD:R_0805_2012Metric_Pad1.20x1.40mm_HandSolder -> Resistor_SMD:R_0603_1608Metric_Pad0.98x0.95mm_HandSolder; LCSC C2930231 -> C21190; Price 0.0017 -> 0.0016
- R20: renamed from R36; value 1k -> 1K
- R22: renamed from R32; value 1k -> 1K
- R24: renamed from R35; value 1k -> 1K
- R25: renamed from R41; value 1k -> 1K
- R3: value 10K -> 4.7K; LCSC C2930231 -> C2960810; Price 0.0017 -> 0.0012
- R9: value 3.3K -> 100k; footprint Resistor_SMD:R_0805_2012Metric_Pad1.20x1.40mm_HandSolder -> Resistor_SMD:R_0603_1608Metric_Pad0.98x0.95mm_HandSolder; LCSC C2907249 -> C14675; Price 0.0020 -> 0.0014
- SW1: footprint Button_Switch_SMD:SW_SPST_CK_RS282G05A3 -> Button_Switch_THT:SW_PUSH_6mm_H5mm
- renumbered C2 to C1, C13 to C12, C19 to C13, C30 to C14, C31 to C15, C37 to C18, C33 to C19, C35 to C20, C26 to C21, C25 to C22, C38 to C23, C39 to C24, C8 to C7, D4 to D2, D5 to D3, J23 to J5, JP4 to JP8, K2 to K1, Q4 to Q2, R2 to R1, R30 to R14, R25 to R15, R38 to R19, R33 to R23, R42 to R26, R8 to R6, R14 to R8, U1 to U2, U9 to U3, U12 to U4, Y2 to Y1, Y1 to Y2
Connections:
- net 12VA is gone; now on net +3.3V: JP5.2 (B)
- net DC_DRV_1 is gone; now on net RLY_DRV: U3.16 (PA6)
- net GNDPWR is gone; now on net GND: C1.2, C10.2, C11.2, C13.2, C4.2, C5.1, Q2.2 (S), R1.2, R19.2, R23.1, R6.2, U2.7 (GND), U2.EPAD (GND), U4.2
- net TMR_CLK is gone; now on net BTN_MODE_1: U3.26 (PB13)
- net TMR_DATA is gone; now on net BTN_MODE_3: U3.28 (PB15)
- net TMR_LOAD is gone; now on net BTN_MODE_2: U3.27 (PB14)
- net VBAT is gone; now on net +3.3V: U3.1 (VBAT)
- net +3.3V: now also C16.1, C5.2, C6.2, C9.2, R13.1, R16.1, R18.1, R3.1, C8.2, D4.2 (A), JP6.1 (A), JP9.1 (A), R17.1, R2.1, U1.2 (VO); no longer C3.2, C9.1, R11.1, R9.1
- net +5V: now also C12.1, C13.1, C3.2, L1.2, R7.1, C2.2, J3.1 (Pin_1), J4.1 (Pin_1), J7.1 (Pin_1), JP4.2 (B), JP6.3 (B), JP9.3 (B), U1.3 (VI); no longer C16.2, C6.2, JP1.2 (B), R13.1, R16.1, R18.1, R21.1
- net +5VA: no longer C12.1, C13.1, C5.2, JP1.1 (A), L1.2, R7.1
- net GND: now also C16.2, C17.1, C18.1, C19.1, C20.1, C23.1, C24.1, C3.1, C6.1, C9.1, R11.2, R21.2, R26.1, SW1.2, U3.23 (VSS), U3.35 (VSS__1), U3.47 (VSS__2), U3.8 (VSSA), U4.3, C2.1, C8.1, J1.2 (Pin_2), J2.2, J3.5 (Pin_5), J4.5 (Pin_5), J6.4 (Pin_4), J7.4 (Pin_4), J9.4 (Pin_4), JP10.1 (A), JP7.1 (A), Q1.2 (S), Q3.2 (S), R27.2, R29.2, R30.2, SW2.1, SW3.1, SW4.1, SW5.5 (B), U1.1 (GND)
- net SEG_CLK: now also J9.2 (Pin_2)
- net SEG_DIO: now also J9.3 (Pin_3)
- net STM_RST: now also SW1.1; no longer SW1.2
- net AUX_1: now reaches U3.18 (PB0)
- net AUX_1: now also J6.2 (Pin_2)
- net AUX_2: now reaches U3.19 (PB1)
- net AUX_2: now also J6.3 (Pin_3)
- net +12V: now reaches JP3.2 (B)
- net +12V: now also C1.1, C4.1, U2.2 (VIN), U2.3 (EN), J10.3 (Pin_3), J11.2 (Pin_2), J2.1
- net BTN_MODE_2: now reaches R16.2
- net BTN_MODE_2: now also SW3.2
- net RLY_DRV: now reaches Q2.1 (G), R19.1
- net at JP8.1 (A), R22.2, R23.2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: now also J10.2 (Pin_2)
- net BTN_MODE_3: now reaches R18.2
- net BTN_MODE_3: now also SW4.2
- net at JP3.1 (A): now also JP5.1 (A), J1.3 (Pin_3), JP4.1 (A); no longer R3.2
- net at J5.4 (Pin_4): now also R9.2
- net BTN_MODE_1: now reaches R13.2
- net BTN_MODE_1: now also SW2.2
- removed net 12V: C1.1, C4.1, JP5.1 (A), U2.2 (VIN), U2.3 (EN)
- net 12V_SEL renamed RLY_NC
- net RLY_NC: now also J12.1 (Pin_1); no longer K1.2
- net BUTTON_1 renamed USER_BTN
- net USER_BTN: now also J1.1 (Pin_1)
- net COM renamed RLY_COM
- net RLY_COM: now also J12.2 (Pin_2), SW5.4 (A)
- net CTRL_DCI1: no longer names the net of U3.46 (PB9)
- net EN_COIN renamed COIN_EN
- net COIN_EN: now also R21.1, Q3.1 (G)
- net ESP_INT renamed I2C_INT
- net I2C_INT: now also J3.4 (Pin_4), J4.4 (Pin_4)
- removed net GNDD: C16.1, C17.1, C18.1, C19.1, C20.1, C23.1, C24.1, C3.1, C6.1, C9.2, R26.1, R3.1, R9.2, SW1.1, U3.23 (VSS), U3.35 (VSS__1), U3.47 (VSS__2), U3.8 (VSSA), U4.3
- net I2C_CONF renamed I2C_CONFG
- net I2C_CONFG: now also JP10.2 (C), R17.2; no longer R11.2
- net LED_P renamed USER_LED
- net USER_LED: now also R11.1, Q1.1 (G)
- net OSCIN: no longer names the net of C22.2, R15.1, Y2.2
- net OSCIN: now also U3.6 (PD1_OSC_OUT); no longer U3.5 (PD0_OSC_IN)
- net OSCOUT: no longer names the net of C21.2, R15.2, Y2.1
- net OSCOUT: now also U3.5 (PD0_OSC_IN); no longer U3.6 (PD1_OSC_OUT)
- net PA11: no longer names the net of U3.32 (PA11)
- net PA12: no longer names the net of U3.33 (PA12)
- net PC14: no longer names the net of C14.2, U3.3 (PC14-OSC32_IN), Y1.2
- net PC15: no longer names the net of C15.2, U3.4 (PC15-OSC32_OUT), Y1.1
- net STM32_BOOT0 renamed STM_BOOT0
- net STM_BOOT0: now also R8.1
- net STM32_BOOT1 renamed STM_BOOT1
- net STM_BOOT1: now also R9.1; no longer R8.1
- net STM32_IN1 renamed COIN_IN
- net STM32_RX renamed STM_RX
- net STM_RX: now also J7.3 (Pin_3)
- net STM32_SCL renamed STM_SCL
- net STM_SCL: now also JP1.1 (A), J3.2 (Pin_2), J4.2 (Pin_2)
- net STM32_SDA renamed STM_SDA
- net STM_SDA: now also J3.3 (Pin_3), J4.3 (Pin_3), JP2.1 (A)
- net STM32_SWCLK: no longer names the net of U3.37 (PA14)
- net STM32_SWDIO: no longer names the net of U3.34 (PA13)
- net STM32_TX renamed STM_TX
- net STM_TX: now also J7.2 (Pin_2)
- net UART_RX1 renamed DBG_LED_B
- net DBG_LED_B: now also D7.2 (A)
- net UART_TX1 renamed DBG_LED_G
- net DBG_LED_G: now also D6.2 (A)
- net WDT_DONE: no longer names the net of U3.17 (PA7)
- new net: J10.1 (Pin_1), JP7.2 (C)
- new net: D7.1 (K), R30.1
- new net: J6.1 (Pin_1), JP9.2 (C)
- new net: JP1.2 (B), R2.2
- new net: JP2.2 (B), R3.2
- new net: J1.4 (Pin_4), Q1.3 (D)
- new net: D6.1 (K), R29.1
- new net: JP7.3 (B), Q3.3 (D)
- new net: J9.1 (Pin_1), JP6.2 (C)
- new net: D4.1 (K), R27.1
- new net GND_OUT: J11.1 (Pin_1), SW5.2 (B), SW5.6 (C)
- new net RLY_NO: J12.3 (Pin_3), K1.2, SW5.3 (C)
- no-connect marks 9 -> 15
Other:
- note added: "7 SEGMENT"
- note added: "BOOT"
- note added: "Configurations"
- note added: "DAISY CONNECT"
- note added: "LED INDICATORS"
- note added: "MICROCONTROLLER"
- note added: "M|S CONFIG"
- note added: "POWER"
- note added: "PROG"
- note added: "RESET"
- note added: "USER BUTTON AND LED + AUX"
- note removed: "3V3 REGULATOR"
- note removed: "CONNECTOR-FOR-SLAVE"
- note removed: "D"
- note removed: "FC4SDCBMF8"
- note removed: "G"
- note removed: "IF THE PCB IS MASTER POPULATE THIS"
- note removed: "ISOLATED POWER"
- note removed: "Output Capacity 5V, 400mA"
- note removed: "PROGRAMMER"
- note removed: "S"
- note removed: "STM32 BLUEPILL"
- note removed: "STM32 CRYSTAL"
- note removed: "Songle Relay SLA-5VDC-SL-C"
- note removed: "TERMINAL BLOCK IO/s"
- note removed: "TIMER CONFIGURATION"
- note removed: "WATCHDOG TIMER"
- note removed: "https://stm32-base.org/boards/STM32F103C8T6-Blue-Pill.html"
- moved on the sheet: C1, C10, C11, C12, C13, C14, C15, C17, C18, C19, C20, C21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
