File: Vendo_main_board/Vendo_main_board/Vendo_main_board.kicad_pcb (KiCad board)
At the start: 4 copper layers, 100 x 80 mm, 121 parts, among them J1 Conn_01x04, J2 Conn_01x03, J3 Screw_Terminal_01x16, J4 Screw_Terminal_01x16, J6 Conn_01x04, K1 SRD-05VDC-SL-C, K2 SRD-05VDC-SL-C, K3 SRD-05VDC-SL-C, K4 SRD-05VDC-SL-C, K5 SRD-05VDC-SL-C, K6 SRD-05VDC-SL-C, K7 SRD-05VDC-SL-C, K8 SRD-05VDC-SL-C, Q1 Q_NMOS_Depletion_GSD, Q2 Q_NMOS_Depletion_GSD, Q3 Q_NMOS_Depletion_GSD, Q4 Q_NMOS_Depletion_GSD, Q5 Q_NMOS_Depletion_GSD, Q6 Q_NMOS_Depletion_GSD, Q7 Q_NMOS_Depletion_GSD, Q8 Q_NMOS_Depletion_GSD, SW1 SW_Push, SW2 SW_Push, U1 B0505S-2WR3, U10 PC817, U11 74HC595, U12 74HC595, U13 PC817, U14 PC817, U15 PC817, U16 PC817, U2 TPL5010, U3 AMS1117-3.3, U4 MAX485E, U5 MAX485E, U6 ESP32-WROOM-32, U7 PC817, U8 PC817, U9 PC817

Commit message: -update scheme and pcb placement
update scheme and footprint
added spade connectors
Parts:
- added C21: 100nF, Capacitor_SMD:C_0603_1608Metric_Pad1.08x0.95mm_HandSolder, F.Cu at (81.2, 107.3)
- added C22: 10uF, Capacitor_SMD:C_0603_1608Metric_Pad1.08x0.95mm_HandSolder, F.Cu at (81.2, 102.2)
- added C23: 100nF, Capacitor_SMD:C_0603_1608Metric_Pad1.08x0.95mm_HandSolder, F.Cu at (87.6, 98.5)
- added C24: 0.1uF, Capacitor_SMD:C_0603_1608Metric, F.Cu at (85.9, 93.8)
- added C25: 0.1uF, Capacitor_SMD:C_0603_1608Metric, F.Cu at (84.3, 93.8)
- added C26: 22uF, Capacitor_SMD:C_0603_1608Metric, F.Cu at (80.6, 93.8)
- added C27: 0.1uF, Capacitor_SMD:C_0603_1608Metric, F.Cu at (80.7, 92.2)
- added C28: 0.1uF, Capacitor_SMD:C_0603_1608Metric, F.Cu at (90.4, 69.5)
- added C29: 100nF, Capacitor_SMD:C_0603_1608Metric_Pad1.08x0.95mm_HandSolder, F.Cu at (103.8, 108.5)
- added C30: 100nF, Capacitor_SMD:C_0603_1608Metric_Pad1.08x0.95mm_HandSolder, F.Cu at (106.3, 94.7)
- added C31: 10uF, Capacitor_SMD:C_0603_1608Metric_Pad1.08x0.95mm_HandSolder, F.Cu at (106.3, 93.1)
- added C32: 10uF, Capacitor_SMD:C_0805_2012Metric_Pad1.18x1.45mm_HandSolder, F.Cu at (271.9, 110.9)
- added C33: 0.1uF, Capacitor_SMD:C_0603_1608Metric, F.Cu at (288.9, 167.1)
- added C34: 10uF, Capacitor_SMD:C_0805_2012Metric_Pad1.18x1.45mm_HandSolder, F.Cu at (271.9, 114.0)
- added C35: 10uF, Capacitor_SMD:C_0805_2012Metric_Pad1.18x1.45mm_HandSolder, F.Cu at (271.9, 117.0)
- added C36: 10uF, Capacitor_SMD:C_0805_2012Metric_Pad1.18x1.45mm_HandSolder, F.Cu at (271.9, 120.0)
- added C37: 10uF, Capacitor_SMD:C_0805_2012Metric_Pad1.18x1.45mm_HandSolder, F.Cu at (271.9, 123.0)
- added C38: 10uF, Capacitor_SMD:C_0805_2012Metric_Pad1.18x1.45mm_HandSolder, F.Cu at (271.9, 126.0)
- added C39: 10uF, Capacitor_SMD:C_0805_2012Metric_Pad1.18x1.45mm_HandSolder, F.Cu at (271.9, 129.0)
- added C40: 10uF, Capacitor_SMD:C_0805_2012Metric_Pad1.18x1.45mm_HandSolder, F.Cu at (271.9, 132.0)
- added C41: 10uF, Capacitor_SMD:C_0805_2012Metric_Pad1.18x1.45mm_HandSolder, F.Cu at (271.9, 135.0)
- added C42: 10uF, Capacitor_SMD:C_0805_2012Metric_Pad1.18x1.45mm_HandSolder, F.Cu at (348.9, 56.9)
- added C43: 0.1uF, Capacitor_SMD:C_0603_1608Metric, F.Cu at (282.0, 61.0)
- added D18: LED, LED_SMD:LED_0805_2012Metric_Pad1.15x1.40mm_HandSolder, F.Cu at (348.9, 78.2)
- added D19: LED, LED_SMD:LED_0805_2012Metric_Pad1.15x1.40mm_HandSolder, F.Cu at (348.9, 81.2)
- added J10: Screw_Terminal_01x03, Connector_JST:JST_EH_B3B-EH-A_1x03_P2.50mm_Vertical, F.Cu at (132.8, 89.6)
- added J11: Screw_Terminal_01x03, Connector_JST:JST_EH_B3B-EH-A_1x03_P2.50mm_Vertical, F.Cu at (132.8, 95.5)
- added J12: Screw_Terminal_01x03, Connector_JST:JST_EH_B3B-EH-A_1x03_P2.50mm_Vertical, F.Cu at (132.8, 101.3)
- added J13: 197084013, InnovKits:Spade Conn4.8mm, F.Cu at (246.0, -4.45)
- added J14: 197084013, InnovKits:Spade Conn4.8mm, F.Cu at (246.0, 0.74)
- added J15: 197084013, InnovKits:Spade Conn4.8mm, F.Cu at (246.0, 5.93)
- added J16: 197084013, InnovKits:Spade Conn4.8mm, F.Cu at (246.0, 11.1)
- added J17: 197084013, InnovKits:Spade Conn4.8mm, F.Cu at (246.0, 16.3)
- added J18: 197084013, InnovKits:Spade Conn4.8mm, F.Cu at (246.0, 21.5)
- added J19: 197084013, InnovKits:Spade Conn4.8mm, F.Cu at (246.0, 26.7)
- added J20: 197084013, InnovKits:Spade Conn4.8mm, F.Cu at (246.0, 31.9)
- added J21: 197084013, InnovKits:Spade Conn4.8mm, F.Cu at (246.0, 37.1)
- added J22: 197084013, InnovKits:Spade Conn4.8mm, F.Cu at (246.0, 42.3)
- added J23: 197084013, InnovKits:Spade Conn4.8mm, F.Cu at (246.0, 47.5)
- added J24: 197084013, InnovKits:Spade Conn4.8mm, F.Cu at (246.0, 52.7)
- added J25: 197084013, InnovKits:Spade Conn4.8mm, F.Cu at (246.0, 57.8)
- added J26: 197084013, InnovKits:Spade Conn4.8mm, F.Cu at (257.4, -4.45)
- added J27: 197084013, InnovKits:Spade Conn4.8mm, F.Cu at (257.4, 0.74)
- added J28: 197084013, InnovKits:Spade Conn4.8mm, F.Cu at (257.4, 5.93)
- added J29: 197084013, InnovKits:Spade Conn4.8mm, F.Cu at (257.4, 11.1)
- added J30: 197084013, InnovKits:Spade Conn4.8mm, F.Cu at (257.4, 16.3)
- added J31: 197084013, InnovKits:Spade Conn4.8mm, F.Cu at (257.4, 21.5)
- added J32: 197084013, InnovKits:Spade Conn4.8mm, F.Cu at (257.4, 26.7)
- added J33: 197084013, InnovKits:Spade Conn4.8mm, F.Cu at (257.4, 31.9)
- added J34: 197084013, InnovKits:Spade Conn4.8mm, F.Cu at (257.4, 37.1)
- added J35: 197084013, InnovKits:Spade Conn4.8mm, F.Cu at (257.4, 42.3)
- added J36: 197084013, InnovKits:Spade Conn4.8mm, F.Cu at (257.4, 47.5)
- added J37: 197084013, InnovKits:Spade Conn4.8mm, F.Cu at (257.4, 52.7)
- added J38: 197084013, InnovKits:Spade Conn4.8mm, F.Cu at (257.4, 57.8)
- added J39: 197084013, InnovKits:Spade Conn4.8mm, F.Cu at (268.9, -4.45)
- added J40: 197084013, InnovKits:Spade Conn4.8mm, F.Cu at (268.9, 0.74)
- added J41: 197084013, InnovKits:Spade Conn4.8mm, F.Cu at (268.9, 5.93)
- added J42: 197084013, InnovKits:Spade Conn4.8mm, F.Cu at (268.9, 11.1)
- added J43: 197084013, InnovKits:Spade Conn4.8mm, F.Cu at (268.9, 16.3)
- added J44: 197084013, InnovKits:Spade Conn4.8mm, F.Cu at (268.9, 21.5)
- added J45: 197084013, InnovKits:Spade Conn4.8mm, F.Cu at (268.9, 26.7)
- added J46: 197084013, InnovKits:Spade Conn4.8mm, F.Cu at (268.9, 31.9)
- added J47: 197084013, InnovKits:Spade Conn4.8mm, F.Cu at (268.9, 37.1)
- added J48: 197084013, InnovKits:Spade Conn4.8mm, F.Cu at (268.9, 42.3)
- added J49: 197084013, InnovKits:Spade Conn4.8mm, F.Cu at (268.9, 47.5)
- added J5: Screw_Terminal_01x03, Connector_JST:JST_EH_B3B-EH-A_1x03_P2.50mm_Vertical, F.Cu at (132.8, 60.4)
- added J50: 197084013, InnovKits:Spade Conn4.8mm, F.Cu at (268.9, 52.7)
- added J51: 197084013, InnovKits:Spade Conn4.8mm, F.Cu at (268.9, 57.8)
- added J52: 197084013, InnovKits:Spade Conn4.8mm, F.Cu at (280.3, -4.45)
- added J53: 197084013, InnovKits:Spade Conn4.8mm, F.Cu at (280.3, 0.74)
- added J54: 197084013, InnovKits:Spade Conn4.8mm, F.Cu at (280.3, 5.93)
- added J55: 197084013, InnovKits:Spade Conn4.8mm, F.Cu at (280.3, 11.1)
- added J56: 197084013, InnovKits:Spade Conn4.8mm, F.Cu at (280.3, 16.3)
- added J57: 197084013, InnovKits:Spade Conn4.8mm, F.Cu at (280.3, 21.5)
- added J58: 197084013, InnovKits:Spade Conn4.8mm, F.Cu at (280.3, 26.7)
- added J59: 197084013, InnovKits:Spade Conn4.8mm, F.Cu at (280.3, 31.9)
- added J60: 197084013, InnovKits:Spade Conn4.8mm, F.Cu at (280.3, 37.1)
- added J61: 197084013, InnovKits:Spade Conn4.8mm, F.Cu at (280.3, 42.3)
- added J62: 197084013, InnovKits:Spade Conn4.8mm, F.Cu at (280.3, 47.5)
- added J63: 197084013, InnovKits:Spade Conn4.8mm, F.Cu at (280.3, 52.7)
- added J64: 197084013, InnovKits:Spade Conn4.8mm, F.Cu at (280.3, 57.8)
- added J65: 197084013, InnovKits:Spade Conn4.8mm, F.Cu at (291.7, -4.45)
- added J66: 197084013, InnovKits:Spade Conn4.8mm, F.Cu at (291.7, 0.74)
- added J67: 197084013, InnovKits:Spade Conn4.8mm, F.Cu at (291.7, 5.93)
- added J68: 197084013, InnovKits:Spade Conn4.8mm, F.Cu at (291.7, 11.1)
- added J69: 197084013, InnovKits:Spade Conn4.8mm, F.Cu at (291.7, 16.3)
- added J7: Screw_Terminal_01x03, Connector_JST:JST_EH_B3B-EH-A_1x03_P2.50mm_Vertical, F.Cu at (132.8, 72.1)
- added J70: 197084013, InnovKits:Spade Conn4.8mm, F.Cu at (291.7, 21.5)
- added J71: 197084013, InnovKits:Spade Conn4.8mm, F.Cu at (291.7, 26.7)
- added J72: 197084013, InnovKits:Spade Conn4.8mm, F.Cu at (291.7, 31.9)
- added J73: 197084013, InnovKits:Spade Conn4.8mm, F.Cu at (291.7, 37.1)
- added J74: 197084013, InnovKits:Spade Conn4.8mm, F.Cu at (291.7, 42.3)
- added J75: 197084013, InnovKits:Spade Conn4.8mm, F.Cu at (291.7, 47.5)
- added J76: 197084013, InnovKits:Spade Conn4.8mm, F.Cu at (291.7, 52.7)
- added J8: Screw_Terminal_01x03, Connector_JST:JST_EH_B3B-EH-A_1x03_P2.50mm_Vertical, F.Cu at (132.8, 77.9)
- added J9: Screw_Terminal_01x03, Connector_JST:JST_EH_B3B-EH-A_1x03_P2.50mm_Vertical, F.Cu at (132.8, 83.8)
- added JP2: SolderJumper_2_Open, Jumper:SolderJumper-2_P1.3mm_Open_Pad1.0x1.5mm, B.Cu at (109.0, 77.6)
- added JP3: SolderJumper_2_Open, Jumper:SolderJumper-2_P1.3mm_Open_Pad1.0x1.5mm, B.Cu at (109.2, 80.6)
- added JP4: SolderJumper_2_Open, Jumper:SolderJumper-2_P1.3mm_Open_RoundedPad1.0x1.5mm, B.Cu at (100.4, 106.1)
- added JP5: SolderJumper_2_Open, Jumper:SolderJumper-2_P1.3mm_Open_RoundedPad1.0x1.5mm, B.Cu at (103.0, 106.1)
- added JP6: SolderJumper_2_Open, Jumper:SolderJumper-2_P1.3mm_Open_RoundedPad1.0x1.5mm, B.Cu at (105.6, 106.1)
- added L1: 5.5uH, InnovKits:744325550, F.Cu at (108.5, 55.3)
- added Q10: ~, footprints:SOT-23-3_L2.9-W1.6-P1.90-LS2.8-BR, F.Cu at (276.3, 152.1)
- added Q11: S8050, Package_TO_SOT_SMD:SOT-23, F.Cu at (281.8, 138.9)
- added Q12: S8050, Package_TO_SOT_SMD:SOT-23, F.Cu at (281.8, 143.6)
- added Q13: ~, footprints:SOT-23-3_L2.9-W1.6-P1.90-LS2.8-BR, F.Cu at (280.8, 147.9)
- added Q14: ~, footprints:SOT-23-3_L2.9-W1.6-P1.90-LS2.8-BR, F.Cu at (280.8, 152.1)
- added Q15: S8050, Package_TO_SOT_SMD:SOT-23, F.Cu at (286.7, 138.9)
- added Q16: S8050, Package_TO_SOT_SMD:SOT-23, F.Cu at (286.7, 143.6)
- added Q17: ~, footprints:SOT-23-3_L2.9-W1.6-P1.90-LS2.8-BR, F.Cu at (285.4, 147.9)
- added Q18: ~, footprints:SOT-23-3_L2.9-W1.6-P1.90-LS2.8-BR, F.Cu at (285.4, 152.1)
- added Q19: Q_NMOS_Depletion_GSD, Package_TO_SOT_SMD:SOT-23-3, F.Cu at (244.2, 62.2)
- added Q20: Q_NMOS_Depletion_GSD, Package_TO_SOT_SMD:SOT-23-3, F.Cu at (244.2, 66.8)
- added Q21: Q_NMOS_Depletion_GSD, Package_TO_SOT_SMD:SOT-23-3, F.Cu at (249.3, 62.2)
- added Q22: Q_NMOS_Depletion_GSD, Package_TO_SOT_SMD:SOT-23-3, F.Cu at (249.3, 66.8)
- added Q23: Q_NMOS_Depletion_GSD, Package_TO_SOT_SMD:SOT-23-3, F.Cu at (254.5, 62.2)
- added Q24: Q_NMOS_Depletion_GSD, Package_TO_SOT_SMD:SOT-23-3, F.Cu at (254.5, 66.8)
- added Q25: Q_NMOS_Depletion_GSD, Package_TO_SOT_SMD:SOT-23-3, F.Cu at (259.6, 62.2)
- added Q26: Q_NMOS_Depletion_GSD, Package_TO_SOT_SMD:SOT-23-3, F.Cu at (259.6, 66.8)
- added Q9: ~, footprints:SOT-23-3_L2.9-W1.6-P1.90-LS2.8-BR, F.Cu at (276.3, 147.9)
- added R100: 10K, Resistor_SMD:R_0603_1608Metric_Pad0.98x0.95mm_HandSolder, F.Cu at (268.8, 71.1)
- added R101: 10K, Resistor_SMD:R_0603_1608Metric_Pad0.98x0.95mm_HandSolder, F.Cu at (268.8, 73.6)
- added R102: 1k, Resistor_SMD:R_0603_1608Metric_Pad0.98x0.95mm_HandSolder, F.Cu at (273.1, 61.0)
- added R103: 1k, Resistor_SMD:R_0603_1608Metric_Pad0.98x0.95mm_HandSolder, F.Cu at (273.1, 63.5)
- added R104: 1k, Resistor_SMD:R_0603_1608Metric_Pad0.98x0.95mm_HandSolder, F.Cu at (273.1, 66.0)
- added R105: 1k, Resistor_SMD:R_0603_1608Metric_Pad0.98x0.95mm_HandSolder, F.Cu at (273.1, 68.6)
- added R106: 180, Resistor_SMD:R_0805_2012Metric_Pad1.20x1.40mm_HandSolder, F.Cu at (277.6, 73.0)
- added R107: 180, Resistor_SMD:R_0805_2012Metric_Pad1.20x1.40mm_HandSolder, F.Cu at (277.6, 76.0)
- added R108: 180, Resistor_SMD:R_0805_2012Metric_Pad1.20x1.40mm_HandSolder, F.Cu at (277.6, 79.0)
- added R109: 180, Resistor_SMD:R_0805_2012Metric_Pad1.20x1.40mm_HandSolder, F.Cu at (277.6, 81.9)
- added R41: 1k, Resistor_SMD:R_0805_2012Metric_Pad1.20x1.40mm_HandSolder, F.Cu at (281.4, 119.8)
- added R42: 1k, Resistor_SMD:R_0805_2012Metric_Pad1.20x1.40mm_HandSolder, F.Cu at (281.4, 122.7)
- added R43: 1k, Resistor_SMD:R_0805_2012Metric_Pad1.20x1.40mm_HandSolder, F.Cu at (281.4, 125.7)
- added R44: 1k, Resistor_SMD:R_0805_2012Metric_Pad1.20x1.40mm_HandSolder, F.Cu at (281.4, 128.6)
- added R45: 1k, Resistor_SMD:R_0805_2012Metric_Pad1.20x1.40mm_HandSolder, F.Cu at (281.4, 131.6)
- added R46: 100k, Resistor_SMD:R_0603_1608Metric_Pad0.98x0.95mm_HandSolder, F.Cu at (276.0, 160.5)
- added R47: 100k, Resistor_SMD:R_0603_1608Metric_Pad0.98x0.95mm_HandSolder, F.Cu at (276.0, 163.0)
- added R48: 100, Resistor_SMD:R_0603_1608Metric_Pad0.98x0.95mm_HandSolder, F.Cu at (276.0, 165.5)
- added R49: 100, Resistor_SMD:R_0603_1608Metric_Pad0.98x0.95mm_HandSolder, F.Cu at (276.0, 168.0)
- added R50: 1k, Resistor_SMD:R_0805_2012Metric_Pad1.20x1.40mm_HandSolder, F.Cu at (286.2, 110.9)
- added R51: 1k, Resistor_SMD:R_0805_2012Metric_Pad1.20x1.40mm_HandSolder, F.Cu at (286.2, 113.9)
- added R52: 1k, Resistor_SMD:R_0805_2012Metric_Pad1.20x1.40mm_HandSolder, F.Cu at (286.2, 116.8)
- added R53: 1k, Resistor_SMD:R_0805_2012Metric_Pad1.20x1.40mm_HandSolder, F.Cu at (286.2, 119.8)
- added R54: 1k, Resistor_SMD:R_0805_2012Metric_Pad1.20x1.40mm_HandSolder, F.Cu at (286.2, 122.7)
- added R55: 1k, Resistor_SMD:R_0805_2012Metric_Pad1.20x1.40mm_HandSolder, F.Cu at (286.2, 125.7)
- added R56: 4.7k, Resistor_SMD:R_0603_1608Metric_Pad0.98x0.95mm_HandSolder, F.Cu at (280.4, 155.5)
- added R57: 4.7k, Resistor_SMD:R_0603_1608Metric_Pad0.98x0.95mm_HandSolder, F.Cu at (280.4, 158.0)
- added R58: 1k, Resistor_SMD:R_0805_2012Metric_Pad1.20x1.40mm_HandSolder, F.Cu at (286.2, 128.6)
- added R59: 1k, Resistor_SMD:R_0805_2012Metric_Pad1.20x1.40mm_HandSolder, F.Cu at (286.2, 131.6)
- added R60: 1k, Resistor_SMD:R_0805_2012Metric_Pad1.20x1.40mm_HandSolder, F.Cu at (290.9, 110.9)
- added R61: 1k, Resistor_SMD:R_0805_2012Metric_Pad1.20x1.40mm_HandSolder, F.Cu at (290.9, 113.9)
- added R62: 100k, Resistor_SMD:R_0603_1608Metric_Pad0.98x0.95mm_HandSolder, F.Cu at (280.4, 160.5)
- added R63: 100k, Resistor_SMD:R_0603_1608Metric_Pad0.98x0.95mm_HandSolder, F.Cu at (280.4, 163.0)
- added R64: 100, Resistor_SMD:R_0603_1608Metric_Pad0.98x0.95mm_HandSolder, F.Cu at (280.4, 165.5)
- added R65: 100, Resistor_SMD:R_0603_1608Metric_Pad0.98x0.95mm_HandSolder, F.Cu at (280.4, 168.0)
- added R66: 1k, Resistor_SMD:R_0805_2012Metric_Pad1.20x1.40mm_HandSolder, F.Cu at (290.9, 116.8)
- added R67: 1k, Resistor_SMD:R_0805_2012Metric_Pad1.20x1.40mm_HandSolder, F.Cu at (290.9, 119.8)
- added R68: 1k, Resistor_SMD:R_0805_2012Metric_Pad1.20x1.40mm_HandSolder, F.Cu at (290.9, 122.7)
- added R69: 1k, Resistor_SMD:R_0805_2012Metric_Pad1.20x1.40mm_HandSolder, F.Cu at (290.9, 125.7)
- added R70: 4.7k, Resistor_SMD:R_0603_1608Metric_Pad0.98x0.95mm_HandSolder, F.Cu at (284.7, 155.5)
- added R71: 4.7k, Resistor_SMD:R_0603_1608Metric_Pad0.98x0.95mm_HandSolder, F.Cu at (284.7, 158.0)
- added R72: 1k, Resistor_SMD:R_0805_2012Metric_Pad1.20x1.40mm_HandSolder, F.Cu at (290.9, 128.6)
- added R73: 1k, Resistor_SMD:R_0805_2012Metric_Pad1.20x1.40mm_HandSolder, F.Cu at (290.9, 131.6)
- added R74: 1k, Resistor_SMD:R_0805_2012Metric_Pad1.20x1.40mm_HandSolder, F.Cu at (295.7, 110.9)
- added R75: 1k, Resistor_SMD:R_0805_2012Metric_Pad1.20x1.40mm_HandSolder, F.Cu at (295.7, 113.9)
- added R76: 1k, Resistor_SMD:R_0805_2012Metric_Pad1.20x1.40mm_HandSolder, F.Cu at (295.7, 116.8)
- added R77: 1k, Resistor_SMD:R_0805_2012Metric_Pad1.20x1.40mm_HandSolder, F.Cu at (295.7, 119.8)
- added R78: 100k, Resistor_SMD:R_0603_1608Metric_Pad0.98x0.95mm_HandSolder, F.Cu at (284.7, 160.5)
- added R79: 100k, Resistor_SMD:R_0603_1608Metric_Pad0.98x0.95mm_HandSolder, F.Cu at (284.7, 163.0)
- added R80: 100, Resistor_SMD:R_0603_1608Metric_Pad0.98x0.95mm_HandSolder, F.Cu at (284.7, 165.5)
- added R81: 100, Resistor_SMD:R_0603_1608Metric_Pad0.98x0.95mm_HandSolder, F.Cu at (284.7, 168.0)
- added R82: 1k, Resistor_SMD:R_0805_2012Metric_Pad1.20x1.40mm_HandSolder, F.Cu at (295.7, 122.7)
- added R83: 1k, Resistor_SMD:R_0805_2012Metric_Pad1.20x1.40mm_HandSolder, F.Cu at (295.7, 125.7)
- added R84: 1k, Resistor_SMD:R_0805_2012Metric_Pad1.20x1.40mm_HandSolder, F.Cu at (295.7, 128.6)
- added R85: 1k, Resistor_SMD:R_0805_2012Metric_Pad1.20x1.40mm_HandSolder, F.Cu at (295.7, 131.6)
- added R86: 180, Resistor_SMD:R_0805_2012Metric_Pad1.20x1.40mm_HandSolder, F.Cu at (277.6, 61.2)
- added R87: 180, Resistor_SMD:R_0805_2012Metric_Pad1.20x1.40mm_HandSolder, F.Cu at (277.6, 64.2)
- added R88: 180, Resistor_SMD:R_0805_2012Metric_Pad1.20x1.40mm_HandSolder, F.Cu at (277.6, 67.2)
- added R89: 180, Resistor_SMD:R_0805_2012Metric_Pad1.20x1.40mm_HandSolder, F.Cu at (277.6, 70.1)
- added R90: 1k, Resistor_SMD:R_0603_1608Metric_Pad0.98x0.95mm_HandSolder, F.Cu at (264.4, 61.0)
- added R91: 1k, Resistor_SMD:R_0603_1608Metric_Pad0.98x0.95mm_HandSolder, F.Cu at (264.4, 63.5)
- added R92: 1k, Resistor_SMD:R_0603_1608Metric_Pad0.98x0.95mm_HandSolder, F.Cu at (264.4, 66.0)
- added R93: 1k, Resistor_SMD:R_0603_1608Metric_Pad0.98x0.95mm_HandSolder, F.Cu at (264.4, 68.6)
- added R94: 10K, Resistor_SMD:R_0603_1608Metric_Pad0.98x0.95mm_HandSolder, F.Cu at (264.4, 71.1)
- added R95: 10K, Resistor_SMD:R_0603_1608Metric_Pad0.98x0.95mm_HandSolder, F.Cu at (264.4, 73.6)
- added R96: 10K, Resistor_SMD:R_0603_1608Metric_Pad0.98x0.95mm_HandSolder, F.Cu at (268.8, 61.0)
- added R97: 10K, Resistor_SMD:R_0603_1608Metric_Pad0.98x0.95mm_HandSolder, F.Cu at (268.8, 63.5)
- added R98: 10K, Resistor_SMD:R_0603_1608Metric_Pad0.98x0.95mm_HandSolder, F.Cu at (268.8, 66.0)
- added R99: 10K, Resistor_SMD:R_0603_1608Metric_Pad0.98x0.95mm_HandSolder, F.Cu at (268.8, 68.6)
- added U17: PC817, InnovKits:APC-817xx-SL_AMB, F.Cu at (251.0, 151.3)
- added U18: PC817, InnovKits:APC-817xx-SL_AMB, F.Cu at (251.0, 157.7)
- added U19: 74HC595, Package_SO:SOIC-16_3.9x9.9mm_P1.27mm, F.Cu at (345.2, 49.7)
- added U20: PC817, InnovKits:APC-817xx-SL_AMB, F.Cu at (347.4, -4.49)
- added U21: PC817, InnovKits:APC-817xx-SL_AMB, F.Cu at (347.4, 1.95)
- added U22: PC817, InnovKits:APC-817xx-SL_AMB, F.Cu at (347.4, 8.38)
- added U23: PC817, InnovKits:APC-817xx-SL_AMB, F.Cu at (347.4, 14.8)
- added U24: PC817, InnovKits:APC-817xx-SL_AMB, F.Cu at (347.4, 21.3)
- added U25: PC817, InnovKits:APC-817xx-SL_AMB, F.Cu at (347.4, 27.7)
- added U26: PC817, InnovKits:APC-817xx-SL_AMB, F.Cu at (347.4, 34.1)
- added U27: PC817, InnovKits:APC-817xx-SL_AMB, F.Cu at (347.4, 40.6)
- added USB1: ~, InnovKits:USB-C-SMD_TYPE-C16PIN, F.Cu at (79.4, 115.0)
- C1: footprint Capacitor_SMD:C_0805_2012Metric_Pad1.18x1.45mm_HandSolder -> Capacitor_SMD:C_1206_3216Metric_Pad1.33x1.80mm_HandSolder
- C10: value 10uF -> 100uF; footprint Capacitor_SMD:C_0805_2012Metric_Pad1.18x1.45mm_HandSolder -> Capacitor_SMD:C_1210_3225Metric_Pad1.33x2.70mm_HandSolder; moved to F.Cu
- C11: value 22uF -> 10uF; footprint Capacitor_SMD:C_0603_1608Metric -> Capacitor_SMD:C_0805_2012Metric_Pad1.18x1.45mm_HandSolder
- C12: value 10uF -> 100nF; footprint Capacitor_SMD:C_0805_2012Metric_Pad1.18x1.45mm_HandSolder -> Capacitor_SMD:C_0603_1608Metric_Pad1.08x0.95mm_HandSolder; moved to F.Cu
- C13: value 0.1uF -> 100nF; footprint Capacitor_SMD:C_0603_1608Metric -> Capacitor_SMD:C_0603_1608Metric_Pad1.08x0.95mm_HandSolder; moved to F.Cu
- C14, C16, C18: value 0.1uF -> 1uF; footprint Capacitor_SMD:C_0603_1608Metric -> Capacitor_SMD:C_0805_2012Metric_Pad1.18x1.45mm_HandSolder
- C15: value 0.1uF -> 470pF; footprint Capacitor_SMD:C_0603_1608Metric -> Capacitor_SMD:C_0603_1608Metric_Pad1.08x0.95mm_HandSolder; moved to F.Cu
- C17: value 10uF -> 10nF; footprint Capacitor_SMD:C_0805_2012Metric_Pad1.18x1.45mm_HandSolder -> Capacitor_SMD:C_0603_1608Metric_Pad1.08x0.95mm_HandSolder
- C19: value 10uF -> 100nF; footprint Capacitor_SMD:C_0805_2012Metric_Pad1.18x1.45mm_HandSolder -> Capacitor_SMD:C_0603_1608Metric_Pad1.08x0.95mm_HandSolder
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Connections:
- C1 pad 1: GNDPWR -> VIN+_NON_ISO
- C1 pad 2: +5VA -> VIN-_REL_IN
- C10 pad 1: GNDD -> +5V
- C10 pad 2: +5V -> GNDD
- C11 pad 1: +3.3V -> GNDD
- C11 pad 2: GNDD -> +5V
- C12 pad 1: GNDD -> +5V
- C12 pad 2: +5V -> GNDD
- C13 pad 1: +5V -> GNDD
- C13 pad 2: GNDD -> +5V
- C14 pad 1: +3.3V -> GND
- C14 pad 2: GNDD -> +5V
- C15 pad 1: +5V -> GND
- C15 pad 2: GNDD -> Net-(U5-CT)
- C16 pad 1: ESP_I0 -> GNDD
- C16 pad 2: GNDD -> Net-(JP3-B)
- C17 pad 2: +5V -> Net-(U6-FB)
- C18 pad 2: +5V -> +3.3V
- C19 pad 2: +5V -> +3.3V
- C2 pad 1: +5VA -> VIN+_NON_ISO
- C2 pad 2: GNDPWR -> VIN-_REL_IN
- C20 pad 2: +5V -> +3.3V
- C3 pad 1: +5V -> Net-(U1-BST)
- C3 pad 2: GNDD -> Net-(U1-SW)
- C4 pad 1: +5V -> Net-(C4-Pad1)
- C4 pad 2: GNDD -> VIN-_REL_IN
- C5 pad 1: GNDD -> Net-(U1-COMP)
- C5 pad 2: +5V -> VIN-_REL_IN
- C6 pad 1: GNDD -> +5VA
- C6 pad 2: +5V -> GND
- C7 pad 1: GNDD -> +5VA
- C7 pad 2: +3.3V -> VIN-_REL_IN
- C8 pad 1: GNDD -> VIN-_REL_IN
- C8 pad 2: ESP_EN -> +5VA
- C9 pad 1: GNDD -> +5VA
- C9 pad 2: ESP_EN -> VIN-_REL_IN
- D1 pad 1: Net-(D1-K) -> VIN-_REL_IN
- D14 pad 1: Net-(D10-K) -> Net-(D14-K)
- D14 pad 2: Net-(D14-A) -> +5VA
- D15 pad 1: Net-(D11-K) -> Net-(D15-K)
- D15 pad 2: Net-(D15-A) -> +5VA
- D2 pad 1: Net-(D2-K) -> /ESP32_MAIN_MCU/ESP_RX
- D3 pad 1: Net-(D3-K) -> /ESP32_MAIN_MCU/ESP_TX
- D6 pad 1: Net-(D2-K) -> Net-(D10-K)
- D6 pad 2: +5VA -> Net-(D6-A)
- D7 pad 1: Net-(D3-K) -> Net-(D11-K)
- D7 pad 2: +5VA -> Net-(D7-A)
- J1 pad 1: ESP_TX -> DC_IN_1_A
- J1 pad 2: ESP_RX -> DC_IN_1_B
- J1 pad 3: ESP_EN -> DC_IN_2_A
- J1 pad 4: ESP_I0 -> DC_IN_2_B
- J2 pad 1: +5V -> DIN_BTN_1
- J2 pad 2: +3.3V -> DIN_BTN_2
- J2 pad 3: GNDD -> DIN_BTN_3
- J3 pad 1: NO8 -> DIN_BTN_5
- J3 pad 10: NO5 -> TB_SCL
- J3 pad 11: COM5 -> +5V
- J3 pad 12: NC5 -> GNDD
- J3 pad 2: COM8 -> DIN_BTN_6
- J3 pad 3: NC8 -> DIN_BTN_7
- J3 pad 4: NO7 -> DIN_BTN_8
- J3 pad 5: COM7 -> unconnected-(J3-Pin_5-Pad5)
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Routing:
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- removed copper zone on B.Cu, net GNDD
- removed copper zone on F.Cu, net GNDD
- removed copper zone on In1.Cu, net GNDD
- removed copper zone on In2.Cu, net GNDD
- removed copper zone on B.Cu, net GNDPWR
- removed copper zone on F.Cu, net GNDPWR
- removed copper zone on In1.Cu, net GNDPWR
- removed copper zone on In2.Cu, net GNDPWR
Other:
- board size 100 x 80 mm -> 145 x 75 mm
- board text removed: "*"
- board text removed: "3V3"
- board text removed: "5V"
- board text removed: "B0"
- board text removed: "COM1"
- board text removed: "COM2"
- board text removed: "COM3"
- board text removed: "COM4"
- board text removed: "COM5"
- board text removed: "COM6"
- board text removed: "COM7"
- board text removed: "COM8"
- board text removed: "EN"
- board text removed: "EXT.LED"
- board text removed: "G"
- board text removed: "M_A"
- board text removed: "M_B"
- board text removed: "NC1"
- board text removed: "NC2"
- board text removed: "NC3"
- board text removed: "NC4"
- board text removed: "NC5"
- board text removed: "NC6"
- board text removed: "NC7"
- board text removed: "NC8"
- board text removed: "NO1"
- board text removed: "NO2"
- board text removed: "NO3"
- board text removed: "NO4"
- board text removed: "NO5"
- board text removed: "NO6"
- board text removed: "NO7"
- board text removed: "NO8"
- board text removed: "RX"
- board text removed: "S_A"
- board text removed: "S_B"
- board text removed: "TX"

Commit message: -update scheme for modular design
-12V to 5V buck
-5V isolation
-3v3 ldo with wdt
-STM32 blue pill
-dip switch 8 pos with 74HC165
-built in type C programmer
-STLINK 1x4 provisioned
-seven segment port with TM1637 (DIO,CLK)
-relay with 10A & 30A provision , spade connector is put on choosing between 12V supply or external supply , as well on the Common of relay for Ground option
-Coin slot with opto, and loadswitch for it supply 3 pin jst for the port
-slave connector 6 pin jst ,i2c ,5V input for slave seperate gnds
-terminal block for 12V selector for ease of wiring for multiple boards
-terminal io blocks are 16 pin
1button and led with ground pair
12V supply for  device and external supply with grnd pair
relay nc,no and com
esp interrup,sda,scl and gnd for iot connection
Parts:
- removed C1, C2: 10uF, Capacitor_SMD:C_1206_3216Metric_Pad1.33x1.80mm_HandSolder
- removed C10, C9: 100uF, Capacitor_SMD:C_1210_3225Metric_Pad1.33x2.70mm_HandSolder
- removed C11, C32, C34, C35, C36, C37, C38, C39, C40, C41, C42, C8: 10uF, Capacitor_SMD:C_0805_2012Metric_Pad1.18x1.45mm_HandSolder
- removed C12, C13, C19, C21, C23, C29, C30: 100nF, Capacitor_SMD:C_0603_1608Metric_Pad1.08x0.95mm_HandSolder
- removed C14, C16, C18: 1uF, Capacitor_SMD:C_0805_2012Metric_Pad1.18x1.45mm_HandSolder
- removed C15: 470pF, Capacitor_SMD:C_0603_1608Metric_Pad1.08x0.95mm_HandSolder
- removed C17: 10nF, Capacitor_SMD:C_0603_1608Metric_Pad1.08x0.95mm_HandSolder
- removed C20, C22, C31: 10uF, Capacitor_SMD:C_0603_1608Metric_Pad1.08x0.95mm_HandSolder
- removed C24, C25, C27, C28, C33, C43: 0.1uF, Capacitor_SMD:C_0603_1608Metric
- removed C26: 22uF, Capacitor_SMD:C_0603_1608Metric
- removed C3: 100nF, Capacitor_SMD:C_0603_1608Metric
- removed C4: 3.3nF, Capacitor_SMD:C_0603_1608Metric
- removed C5: 56pF, Capacitor_SMD:C_0603_1608Metric
- removed C6, C7: 22uF, Capacitor_SMD:C_1210_3225Metric
- removed D1, D16, D17, D18, D19, D2, D3, D4, D5, D6, D7: LED, LED_SMD:LED_0805_2012Metric_Pad1.15x1.40mm_HandSolder
- removed D10, D11, D12, D13, D14, D15, D8, D9: 1N4001, Diode_SMD:D_SOD-123F
- removed H1, H2, H3, H4: MountingHole, MountingHole:MountingHole_3.2mm_M3
- removed J1, J2, J3, J4: Screw_Terminal_01x12, TerminalBlock_Phoenix:TerminalBlock_Phoenix_MKDS-1,5-12-5.08_1x12_P5.08mm_Horizontal
- removed J10, J11, J12, J5, J6, J7, J8, J9: Screw_Terminal_01x03, Connector_JST:JST_EH_B3B-EH-A_1x03_P2.50mm_Vertical
- removed J13, J14, J15, J16, J17, J18, J19, J20, J21, J22, J23, J24, J25, J26, J27, J28, J29, J30, J31, J32, J33, J34, J35, J36, J37, J38, J39, J40, J41, J42, J43, J44, J45, J46, J47, J48, J49, J50, J51, J52, J53, J54, J55, J56, J57, J58, J59, J60, J61, J62, J63, J64, J65, J66, J67, J68, J69, J70, J71, J72, J73, J74, J75, J76: 197084013, InnovKits:Spade Conn4.8mm
- removed JP1, JP2, JP3: SolderJumper_2_Open, Jumper:SolderJumper-2_P1.3mm_Open_Pad1.0x1.5mm
- removed JP4, JP5, JP6: SolderJumper_2_Open, Jumper:SolderJumper-2_P1.3mm_Open_RoundedPad1.0x1.5mm
- removed K1, K2, K3, K4, K5, K6, K7, K8: SRD-05VDC-SL-C, Relay_THT:Relay_SPDT_SANYOU_SRD_Series_Form_C
- removed L1: 5.5uH, InnovKits:744325550
- removed Q1, Q2: BSS138, Package_TO_SOT_SMD:SOT-23
- removed Q10, Q13, Q14, Q17, Q18, Q5, Q6, Q9: ~, footprints:SOT-23-3_L2.9-W1.6-P1.90-LS2.8-BR
- removed Q11, Q12, Q15, Q16, Q3, Q4, Q7, Q8: S8050, Package_TO_SOT_SMD:SOT-23
- removed Q19, Q20, Q21, Q22, Q23, Q24, Q25, Q26: Q_NMOS_Depletion_GSD, Package_TO_SOT_SMD:SOT-23-3
- removed R1: 200k, Resistor_SMD:R_0603_1608Metric_Pad0.98x0.95mm_HandSolder
- removed R10: 3.3K, Resistor_SMD:R_0805_2012Metric_Pad1.20x1.40mm_HandSolder
- removed R100, R101, R11, R12, R6, R9, R94, R95, R96, R97, R98, R99: 10K, Resistor_SMD:R_0603_1608Metric_Pad0.98x0.95mm_HandSolder
- removed R102, R103, R104, R105, R90, R91, R92, R93: 1k, Resistor_SMD:R_0603_1608Metric_Pad0.98x0.95mm_HandSolder
- removed R106, R107, R108, R109, R86, R87, R88, R89: 180, Resistor_SMD:R_0805_2012Metric_Pad1.20x1.40mm_HandSolder
- removed R13: 1K, Resistor_SMD:R_0603_1608Metric_Pad0.98x0.95mm_HandSolder
- removed R14, R15, R16, R17, R18, R19, R20, R21: 4.7K, Resistor_SMD:R_0603_1608Metric_Pad0.98x0.95mm_HandSolder
- removed R2: 14k, Resistor_SMD:R_0603_1608Metric_Pad0.98x0.95mm_HandSolder
- removed R22, R23, R24, R25, R28, R29, R34, R35, R36, R37, R40, R41, R42, R43, R44, R45, R50, R51, R52, R53, R54, R55, R58, R59, R60, R61, R66, R67, R68, R69, R72, R73, R74, R75, R76, R77, R82, R83, R84, R85: 1k, Resistor_SMD:R_0805_2012Metric_Pad1.20x1.40mm_HandSolder
- removed R26, R27, R38, R39, R56, R57, R70, R71: 4.7k, Resistor_SMD:R_0603_1608Metric_Pad0.98x0.95mm_HandSolder
- removed R3: 147k, Resistor_SMD:R_0603_1608Metric_Pad0.98x0.95mm_HandSolder
- removed R30, R31, R46, R47, R62, R63, R78, R79: 100k, Resistor_SMD:R_0603_1608Metric_Pad0.98x0.95mm_HandSolder
- removed R32, R33, R48, R49, R64, R65, R80, R81: 100, Resistor_SMD:R_0603_1608Metric_Pad0.98x0.95mm_HandSolder
- removed R4: 28k, Resistor_SMD:R_0603_1608Metric_Pad0.98x0.95mm_HandSolder
- removed R5: 10k, Resistor_SMD:R_0603_1608Metric_Pad0.98x0.95mm_HandSolder
- removed R7: 40.2K, Resistor_SMD:R_0603_1608Metric_Pad0.98x0.95mm_HandSolder
- removed R8: 100K, Resistor_SMD:R_0603_1608Metric_Pad0.98x0.95mm_HandSolder
- removed SW1, SW2: SW_Push, Button_Switch_SMD:SW_SPST_CK_RS282G05A3
- removed U1: AP64350SP-13, InnovKits:AP64350SP-13-L
- removed U10, U19: 74HC595, Package_SO:SOIC-16_3.9x9.9mm_P1.27mm
- removed U11, U12, U13, U14, U15, U16, U17, U18, U20, U21, U22, U23, U24, U25, U26, U27: PC817, InnovKits:APC-817xx-SL_AMB
- removed U2: B0505S-2WR3, InnovKits:B_S-2WR2_MNS
- removed U3: TPL5010, Package_TO_SOT_SMD:SOT-23-6
- removed U4: 74AHCT1G125, Package_TO_SOT_SMD:SOT-23-5_HandSoldering
- removed U5: TPS22917DBV, Package_TO_SOT_SMD:SOT-23-6
- removed U6: TPS73733DCQR, Package_TO_SOT_SMD:SOT-223-6
- removed U7: CH340C, Package_SO:SOP-16_4.4x10.4mm_P1.27mm
- removed U8: ESP32-WROOM-32, RF_Module:ESP32-WROOM-32
- removed U9: MCP23017_SO, Package_SO:SOIC-28W_7.5x17.9mm_P1.27mm
- removed USB1: ~, InnovKits:USB-C-SMD_TYPE-C16PIN
Other:
- board outline removed

Commit message: -pcb , update scheme tweak
-pcb placement
-remove USB prog related , no need we have ftdi stlink
Parts:
- added C1: 22uF, Capacitor_SMD:C_0603_1608Metric, F.Cu at (198.0, 54.3)
- added C10: 3.3nF, Capacitor_SMD:C_0603_1608Metric, B.Cu at (197.1, 53.2)
- added C11: 56pF, Capacitor_SMD:C_0603_1608Metric, B.Cu at (200.3, 53.2)
- added C12: 100uF, Capacitor_SMD:C_1210_3225Metric_Pad1.33x2.70mm_HandSolder, F.Cu at (209.4, 50.7)
- added C13: 22uF, Capacitor_SMD:C_1210_3225Metric, B.Cu at (206.5, 63.0)
- added C16: 10uF, Capacitor_SMD:C_0805_2012Metric_Pad1.18x1.45mm_HandSolder, F.Cu at (209.7, 54.4)
- added C17: 1uF, Capacitor_SMD:C_0805_2012Metric_Pad1.18x1.45mm_HandSolder, F.Cu at (192.6, 56.1)
- added C18: 100nF, Capacitor_SMD:C_0603_1608Metric_Pad1.08x0.95mm_HandSolder, F.Cu at (194.4, 58.0)
- added C19: 22uF, Capacitor_SMD:C_1210_3225Metric, B.Cu at (206.5, 58.2)
- added C2: 10uF, Capacitor_SMD:C_1206_3216Metric_Pad1.33x1.80mm_HandSolder, B.Cu at (197.6, 43.2)
- added C20: 10uF, Capacitor_SMD:C_0603_1608Metric_Pad1.08x0.95mm_HandSolder, F.Cu at (195.3, 55.2)
- added C21: 100nF, Capacitor_SMD:C_0603_1608Metric_Pad1.08x0.95mm_HandSolder, F.Cu at (189.0, 70.7)
- added C22: 100nF, Capacitor_SMD:C_0603_1608Metric_Pad1.08x0.95mm_HandSolder, F.Cu at (191.8, 74.5)
- added C25: 20pF, Capacitor_SMD:C_0603_1608Metric, F.Cu at (200.7, 88.4)
- added C26: 20pF, Capacitor_SMD:C_0603_1608Metric, F.Cu at (209.2, 88.4)
- added C3: 22uF, Capacitor_SMD:C_0603_1608Metric, F.Cu at (193.0, 54.3)
- added C30: 20pF, Capacitor_SMD:C_0603_1608Metric, F.Cu at (193.0, 77.4)
- added C31: 20pF, Capacitor_SMD:C_0603_1608Metric, F.Cu at (198.8, 77.5)
- added C32: 10uF, Capacitor_SMD:C_0805_2012Metric_Pad1.18x1.45mm_HandSolder, F.Cu at (209.0, 79.6)
- added C33: 100nF, Capacitor_SMD:C_0603_1608Metric_Pad1.08x0.95mm_HandSolder, F.Cu at (209.5, 66.5)
- added C34: 100nF, Capacitor_SMD:C_0603_1608Metric_Pad1.08x0.95mm_HandSolder, F.Cu at (210.9, 79.7)
- added C35: 100nF, Capacitor_SMD:C_0603_1608Metric_Pad1.08x0.95mm_HandSolder, F.Cu at (196.1, 72.8)
- added C36: 100nF, Capacitor_SMD:C_0603_1608Metric_Pad1.08x0.95mm_HandSolder, B.Cu at (206.2, 125.6)
- added C37: 100nF, Capacitor_SMD:C_0603_1608Metric_Pad1.08x0.95mm_HandSolder, B.Cu at (223.3, 37.0)
- added C38: 100nF, Capacitor_SMD:C_0603_1608Metric_Pad1.08x0.95mm_HandSolder, F.Cu at (205.7, 76.1)
- added C39: 100nF, Capacitor_SMD:C_0603_1608Metric_Pad1.08x0.95mm_HandSolder, F.Cu at (199.3, 64.1)
- added C4: 10uF, Capacitor_SMD:C_1206_3216Metric_Pad1.33x1.80mm_HandSolder, B.Cu at (197.6, 40.8)
- added C40: 10uF, Capacitor_SMD:C_0805_2012Metric_Pad1.18x1.45mm_HandSolder, B.Cu at (216.3, 119.3)
- added C5: 10uF, Capacitor_SMD:C_0805_2012Metric_Pad1.18x1.45mm_HandSolder, F.Cu at (209.7, 44.5)
- added C6: 1uF, Capacitor_SMD:C_0805_2012Metric_Pad1.18x1.45mm_HandSolder, F.Cu at (198.0, 56.1)
- added C7: 100uF, Capacitor_SMD:C_1210_3225Metric_Pad1.33x2.70mm_HandSolder, F.Cu at (209.4, 40.9)
- added C8: 100nF, Capacitor_SMD:C_0603_1608Metric_Pad1.08x0.95mm_HandSolder, B.Cu at (194.2, 48.0)
- added C9: 100nF, Capacitor_SMD:C_0603_1608Metric_Pad1.08x0.95mm_HandSolder, F.Cu at (190.7, 59.1)
- added D1: LED, LED_SMD:LED_0805_2012Metric_Pad1.15x1.40mm_HandSolder, F.Cu at (192.9, 40.7)
- added D2: LED, LED_SMD:LED_0805_2012Metric_Pad1.15x1.40mm_HandSolder, F.Cu at (193.1, 43.3)
- added D4: LED, LED_SMD:LED_0805_2012Metric_Pad1.15x1.40mm_HandSolder, F.Cu at (188.7, 122.1)
- added D5: 1N4001, Diode_SMD:D_SOD-123F, B.Cu at (211.3, 93.5)
- added H1: MountingHole, MountingHole:MountingHole_3.2mm_M3, F.Cu at (225.0, 41.8)
- added H2: MountingHole, MountingHole:MountingHole_3.2mm_M3, F.Cu at (224.9, 120.6)
- added H3: MountingHole, MountingHole:MountingHole_3.2mm_M3, F.Cu at (183.0, 120.7)
- added H4: MountingHole, MountingHole:MountingHole_3.2mm_M3, F.Cu at (183.0, 41.8)
- added J1: STLINK, Connector_PinHeader_2.54mm:PinHeader_1x04_P2.54mm_Vertical, F.Cu at (182.2, 55.8)
- added J10: Screw_Terminal_01x04, TerminalBlock_MetzConnect:TerminalBlock_MetzConnect_Type055_RT01504HDWU_1x04_P5.00mm_Horizontal, F.Cu at (201.6, 33.8)
- added J11: Screw_Terminal_01x04, TerminalBlock_MetzConnect:TerminalBlock_MetzConnect_Type055_RT01504HDWU_1x04_P5.00mm_Horizontal, F.Cu at (186.6, 128.8)
- added J12: Screw_Terminal_01x02, TerminalBlock_MetzConnect:TerminalBlock_MetzConnect_Type073_RT02602HBLU_1x02_P5.08mm_Horizontal, F.Cu at (225.9, 96.4)
- added J13: Screw_Terminal_01x02, TerminalBlock_MetzConnect:TerminalBlock_MetzConnect_Type073_RT02602HBLU_1x02_P5.08mm_Horizontal, F.Cu at (181.9, 91.3)
- added J14: 197084013, InnovKits:Spade Conn4.8mm, F.Cu at (181.9, 109.1)
- added J15: 197084013, InnovKits:Spade Conn4.8mm, F.Cu at (181.9, 112.1)
- added J16: 197084013, InnovKits:Spade Conn4.8mm, F.Cu at (181.9, 102.2)
- added J17: 197084013, InnovKits:Spade Conn4.8mm, F.Cu at (181.9, 115.1)
- added J18: 197084013, InnovKits:Spade Conn4.8mm, F.Cu at (181.9, 105.1)
- added J19: FTDI, Connector_PinHeader_2.54mm:PinHeader_1x04_P2.54mm_Vertical, F.Cu at (185.9, 55.8)
- added J2: Conn_01x02_Pin, Connector_PinHeader_2.54mm:PinHeader_1x02_P2.54mm_Vertical, F.Cu at (217.2, 83.9)
- added J21: Conn_01x04_Pin, Connector_PinHeader_2.54mm:PinHeader_1x04_P2.54mm_Vertical, F.Cu at (182.2, 59.8)
- added J23: BOOT, Connector_PinSocket_2.54mm:PinSocket_2x03_P2.54mm_Vertical, F.Cu at (192.9, 84.0)
- added J5: Screw_Terminal_01x03, TerminalBlock_MetzConnect:TerminalBlock_MetzConnect_Type073_RT02603HBLU_1x03_P5.08mm_Horizontal, F.Cu at (226.0, 113.1)
- added J6: Conn_01x06_Pin, Connector_JST:JST_EH_B6B-EH-A_1x06_P2.50mm_Vertical, F.Cu at (225.6, 84.8)
- added J7: Conn_01x06_Pin, Connector_JST:JST_EH_B6B-EH-A_1x06_P2.50mm_Vertical, F.Cu at (182.2, 72.3)
- added J8: Screw_Terminal_01x04, TerminalBlock_MetzConnect:TerminalBlock_MetzConnect_Type055_RT01504HDWU_1x04_P5.00mm_Horizontal, F.Cu at (206.7, 128.8)
- added J9: Screw_Terminal_01x04, TerminalBlock_MetzConnect:TerminalBlock_MetzConnect_Type055_RT01504HDWU_1x04_P5.00mm_Horizontal, F.Cu at (221.7, 33.8)
- added JP1: SolderJumper_2_Open, Jumper:SolderJumper-2_P1.3mm_Open_RoundedPad1.0x1.5mm, B.Cu at (209.1, 47.4)
- added JP3: SolderJumper_2_Open, Jumper:SolderJumper-2_P1.3mm_Open_RoundedPad1.0x1.5mm, F.Cu at (190.2, 61.6)
- added JP4: SolderJumper_2_Open, Jumper:SolderJumper-2_P1.3mm_Open_RoundedPad1.0x1.5mm, B.Cu at (214.9, 104.6)
- added JP5: SolderJumper_2_Open, Jumper:SolderJumper-2_P1.3mm_Open_RoundedPad1.0x1.5mm, B.Cu at (225.3, 116.5)
- added K1: SRD-05VDC-SL-C, Relay_THT:Relay_SPDT_SANYOU_SRD_Series_Form_C, F.Cu at (205.1, 102.1)
- added K2: ~, InnovKits:RELAY-TH_SLA-XXVDC-SL-C, F.Cu at (204.1, 108.1)
- added L1: 6.8uH, InnovKits:IND-SMD_L11.5-W10.0_FXL1040, B.Cu at (197.9, 60.2)
- added Q3: S8050, Package_TO_SOT_SMD:SOT-23, B.Cu at (218.9, 115.6)
- added Q4: Q_NMOS_Depletion_GSD, Package_TO_SOT_SMD:SOT-23-3, B.Cu at (215.1, 90.2)
- added Q5: ~, footprints:SOT-23-3_L2.9-W1.6-P1.90-LS2.8-BR, B.Cu at (220.9, 118.8)
- added R1: 1k, Resistor_SMD:R_0603_1608Metric_Pad0.98x0.95mm_HandSolder, F.Cu at (196.8, 43.3)
- added R10: 10K, Resistor_SMD:R_0805_2012Metric_Pad1.20x1.40mm_HandSolder, F.Cu at (196.8, 40.7)
- added R11: 1k, Resistor_SMD:R_0603_1608Metric_Pad0.98x0.95mm_HandSolder, F.Cu at (214.6, 83.7)
- added R12: 1k, Resistor_SMD:R_0603_1608Metric_Pad0.98x0.95mm_HandSolder, F.Cu at (189.0, 74.1)
- added R13: 10K, Resistor_SMD:R_0805_2012Metric_Pad1.20x1.40mm_HandSolder, F.Cu at (215.9, 66.5)
- added R14: 100k, Resistor_SMD:R_0603_1608Metric_Pad0.98x0.95mm_HandSolder, F.Cu at (195.5, 87.0)
- added R15: 100k, Resistor_SMD:R_0603_1608Metric_Pad0.98x0.95mm_HandSolder, F.Cu at (188.0, 85.2)
- added R16: 10K, Resistor_SMD:R_0805_2012Metric_Pad1.20x1.40mm_HandSolder, F.Cu at (215.9, 64.0)
- added R18: 10K, Resistor_SMD:R_0805_2012Metric_Pad1.20x1.40mm_HandSolder, F.Cu at (215.9, 61.5)
- added R19: 10K, Resistor_SMD:R_0805_2012Metric_Pad1.20x1.40mm_HandSolder, F.Cu at (215.9, 58.9)
- added R2: 200k, Resistor_SMD:R_0603_1608Metric_Pad0.98x0.95mm_HandSolder, B.Cu at (201.0, 42.6)
- added R21: 10K, Resistor_SMD:R_0805_2012Metric_Pad1.20x1.40mm_HandSolder, F.Cu at (215.9, 56.4)
- added R23: 10K, Resistor_SMD:R_0805_2012Metric_Pad1.20x1.40mm_HandSolder, F.Cu at (215.9, 53.9)
- added R24: 10K, Resistor_SMD:R_0805_2012Metric_Pad1.20x1.40mm_HandSolder, F.Cu at (215.9, 51.3)
- added R25: 1M, Resistor_SMD:R_0603_1608Metric, F.Cu at (203.9, 80.9)
- added R26: 10K, Resistor_SMD:R_0805_2012Metric_Pad1.20x1.40mm_HandSolder, F.Cu at (215.9, 48.8)
- added R29: 1k, Resistor_SMD:R_0603_1608Metric_Pad0.98x0.95mm_HandSolder, B.Cu at (209.6, 125.6)
- added R3: 10K, Resistor_SMD:R_0603_1608Metric_Pad0.98x0.95mm_HandSolder, F.Cu at (187.2, 60.9)
- added R30: 100K, Resistor_SMD:R_0603_1608Metric_Pad0.98x0.95mm_HandSolder, B.Cu at (219.9, 37.0)
- added R31: 10K, Resistor_SMD:R_0805_2012Metric_Pad1.20x1.40mm_HandSolder, B.Cu at (198.0, 90.3)
- added R32: 1k, Resistor_SMD:R_0603_1608Metric_Pad0.98x0.95mm_HandSolder, B.Cu at (216.9, 112.5)
- added R33: 1k, Resistor_SMD:R_0603_1608Metric_Pad0.98x0.95mm_HandSolder, B.Cu at (220.3, 112.5)
- added R34: 4.7k, Resistor_SMD:R_0603_1608Metric_Pad0.98x0.95mm_HandSolder, B.Cu at (216.1, 115.5)
- added R35: 1k, Resistor_SMD:R_0603_1608Metric_Pad0.98x0.95mm_HandSolder, B.Cu at (218.9, 110.8)
- added R36: 1k, Resistor_SMD:R_0603_1608Metric_Pad0.98x0.95mm_HandSolder, F.Cu at (188.7, 118.5)
- added R37: 1k, Resistor_SMD:R_0603_1608Metric_Pad0.98x0.95mm_HandSolder, F.Cu at (220.4, 122.5)
- added R38: 10K, Resistor_SMD:R_0805_2012Metric_Pad1.20x1.40mm_HandSolder, B.Cu at (212.0, 90.3)
- added R39: 100k, Resistor_SMD:R_0603_1608Metric_Pad0.98x0.95mm_HandSolder, B.Cu at (218.2, 119.2)
- added R4: 40.2K, Resistor_SMD:R_0603_1608Metric_Pad0.98x0.95mm_HandSolder, F.Cu at (187.2, 62.4)
- added R40: 100, Resistor_SMD:R_0603_1608Metric_Pad0.98x0.95mm_HandSolder, B.Cu at (221.7, 115.0)
- added R41: 1k, Resistor_SMD:R_0603_1608Metric_Pad0.98x0.95mm_HandSolder, B.Cu at (219.0, 97.4)
- added R42: 1k, Resistor_SMD:R_0603_1608Metric_Pad0.98x0.95mm_HandSolder, B.Cu at (219.0, 95.8)
- added R5: 14k, Resistor_SMD:R_0603_1608Metric_Pad0.98x0.95mm_HandSolder, B.Cu at (198.7, 53.3)
- added R6: 100K, Resistor_SMD:R_0603_1608Metric_Pad0.98x0.95mm_HandSolder, F.Cu at (197.6, 59.5)
- added R7: 147k, Resistor_SMD:R_0603_1608Metric_Pad0.98x0.95mm_HandSolder, B.Cu at (202.1, 51.6)
- added R8: 28k, Resistor_SMD:R_0603_1608Metric_Pad0.98x0.95mm_HandSolder, B.Cu at (202.1, 48.2)
- added R9: 3.3K, Resistor_SMD:R_0805_2012Metric_Pad1.20x1.40mm_HandSolder, F.Cu at (190.2, 53.1)
- added SW1: SW_Push, Button_Switch_SMD:SW_SPST_CK_RS282G05A3, F.Cu at (191.9, 68.7)
- added SW2: SW_DIP_x08, Button_Switch_THT:SW_DIP_SPSTx08_Slide_9.78x22.5mm_W7.62mm_P2.54mm, F.Cu at (226.9, 66.5)
- added TP1: TestPoint, TestPoint:TestPoint_Pad_D1.0mm, F.Cu at (188.1, 64.3)
- added TP2: TestPoint, TestPoint:TestPoint_Pad_D1.0mm, F.Cu at (199.5, 60.4)
- added U1: AP64350SP-13, InnovKits:AP64350SP-13-L, B.Cu at (198.4, 48.1)
- added U10: 74HC165, InnovKits:SOIC-16_L9.9-W3.9-P1.27-LS6.0-BL, F.Cu at (216.0, 75.9)
- added U11: PC817, InnovKits:APC-817xx-SL_AMB, B.Cu at (205.1, 90.3)
- added U12: PC817, InnovKits:APC-817xx-SL_AMB, B.Cu at (219.0, 104.1)
- added U2: AMS1117-3.3, Package_TO_SOT_SMD:SOT-223-3_TabPin2, F.Cu at (194.9, 49.0)
- added U3: B0505S-2WR3, InnovKits:B_S-2WR2_MNS, F.Cu at (206.5, 41.4)
- added U4: TPL5010, Package_TO_SOT_SMD:SOT-23-6, F.Cu at (194.6, 61.3)
- added U9: STM32F103C8T6, InnovKits:LQFP-48_L7.0-W7.0-P0.50-LS9.0-BL, F.Cu at (203.3, 70.1)
- added Y1: 8MHz, InnovKits:HC-49S_L11.4-W4.9-LS13.4, F.Cu at (204.9, 84.8)
- added Y2: 32.768kHz, InnovKits:OSC-SMD_L3.2-W1.5, F.Cu at (195.9, 77.5)
Routing:
- net 12V: track 0.00 -> 99.0 mm, vias 0 -> 1
- net /EXT: track 0.00 -> 86.9 mm
Other:
- board outline added: 49 x 99 mm
- copper layers 4 -> 2
