File: Vendo_main_board/Vendo_main_board/Vendo_main_board.kicad_pcb (KiCad board)
At the start: 2 copper layers, 60 x 100 mm, 117 parts, among them J1 Screw_Terminal_01x04, J10 Screw_Terminal_01x03, J11 Screw_Terminal_01x02, J12 Screw_Terminal_01x03, J2 Barrel_Jack_MountingPin, J3 Conn_01x05_Pin, J4 Conn_01x05_Pin, J5 BOOT, J6 Screw_Terminal_01x04, J7 FTDI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

Commit message: -pcb minor edit
-copper pour on nc,no and com for thick trace
- via flood on regulator and buck
- via stich for mcu side
- thicker trace for 12V bottom part
Routing:
- net GND: track 93.9 -> 133.3 mm, vias 98 -> 316
- added copper zone on B.Cu, net RLY_COM
- added copper zone on F.Cu, net RLY_NC
- added copper zone on F.Cu, net RLY_NO
Other:
- outline, holes or cut-outs redrawn

Commit message: -repush
Changed lines of the file:
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@@
 	)
 	(segment
-		(start 234.355 29.53)
-		(end 211.91 29.53)
+		(start 212.06 29.53)
+		(end 199.92 41.67)
 		(width 0.7)
 		(layer "B.Cu")
@@
 	)
 	(segment
-		(start 211.91 29.53)
-		(end 199.92 41.52)
+		(start 199.92 41.67)
+		(end 199.92 117.64)
+		(width 0.7)
+		(layer "B.Cu")
+		(net 1)
+	)
+	(segment
+		(start 206.57 120.9)
+		(end 206.57 124.66)
+		(width 0.7)
+		(layer "B.Cu")
+		(net 1)
+	)
+	(segment
+		(start 234.355 29.53)
+		(end 212.06 29.53)
+		(width 0.7)
+		(layer "B.Cu")
+		(net 1)
+	)
+	(segment
+		(start 244.3625 124.5175)
+		(end 244.3625 122.3025)
+		(width 0.7)
+		(layer "B.Cu")
+		(net 1)
+	)
+	(segment
+		(start 243.02 125.86)
+		(end 244.3625 124.5175)
+		(width 0.7)
+		(layer "B.Cu")
+		(net 1)
+	)
+	(segment
+		(start 239.935 35.11)
+		(end 234.355 29.53)
 		(width 0.7)
 		(layer "B.Cu")
@@
 	)
 	(segment
-		(start 239.935 35.11)
-		(end 234.355 29.53)
+		(start 204.51 118.84)
+		(end 206.57 120.9)
 		(width 0.7)
 		(layer "B.Cu")
@@
 	)
 	(segment
-		(start 204.51 118.84)
-		(end 206.57 120.9)
-		(width 0.7)
-		(layer "B.Cu")
-		(net 1)
-	)
-	(segment
-		(start 206.57 120.9)
-		(end 206.57 124.66)
-		(width 0.7)
-		(layer "B.Cu")
-		(net 1)
-	)
-	(segment
-		(start 199.92 41.52)
-		(end 199.92 117.64)
-		(width 0.7)
-		(layer "B.Cu")
-		(net 1)
-	)
-	(segment
-		(start 244.3625 124.5175)
-		(end 244.3625 122.3025)
+		(start 206.57 124.66)
+		(end 207.77 125.86)
 		(width 0.7)
 		(layer "B.Cu")
@@
 		(width 0.7)
 		(layer "B.Cu")
-		(net 1)
-	)
-	(segment
-		(start 206.57 124.66)
-		(end 207.77 125.86)
-		(width 0.7)
-		(layer "B.Cu")
-		(net 1)
-	)
-	(segment
-		(start 243.02 125.86)
-		(end 244.3625 124.5175)
-		(width 0.7)
-		(layer "B.Cu")
