File: seven segment/seven segment.kicad_sch (KiCad schematic)
At the start: 7 parts, among them J3 Conn_01x08_Pin, J4 Conn_01x04_Pin, U8 TM1637

Commit message: -repush
Parts:
- removed J3: Conn_01x08_Pin, Connector_PinHeader_1.00mm:PinHeader_1x08_P1.00mm_Vertical, symbol Connector:Conn_01x08_Pin
- removed J4: Conn_01x04_Pin, Connector_PinHeader_2.54mm:PinHeader_1x04_P2.54mm_Vertical, symbol Connector:Conn_01x04_Pin
- added U2: CC56-12EWA, Display_7Segment:CA56-12EWA, symbol Display_Character:CC56-12EWA
Connections:
- net GRID1: now also U2.12 (CC1)
- net GRID2: now also U2.9 (CC2)
- net GRID3: now also U2.8 (CC3)
- net GRID4: now also U2.6 (CC4)
- net SEG1/KS1: now also U2.11 (a)
- net SEG2/KS2: now also U2.7 (b)
- net SEG3/KS3: now also U2.4 (c)
- net SEG4/KS4: now also U2.2 (d)
- net SEG5/KS5: now also U2.1 (e)
- net SEG6/KS6: now also U2.10 (f)
- net SEG7/KS7: now also U2.5 (g)
- net SEG8/KS8: now also U2.3 (DPX)
Changed lines of the file:
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@@
 	)
 	(label "SEG8/KS8"
-		(at 81.6231 59.6749 0)
-		(effects
-			(font
-				(size 1.27 1.27)
-			)
-			(justify left bottom)
+		(at 194.183 64.9738 180)
+		(effects
+			(font
+				(size 1.27 1.27)
+			)
+			(justify right bottom)
 		)
 	)
@@
 	)
 	(label "GRID1"
-		(at 81.6231 69.7762 0)
+		(at 250.063 57.3538 0)
 		(effects
 			(font
@@
 	)
 	(label "SEG4/KS4"
-		(at 81.6231 49.5149 0)
-		(effects
-			(font
-				(size 1.27 1.27)
-			)
-			(justify left bottom)
+		(at 194.183 54.8138 180)
+		(effects
+			(font
+				(size 1.27 1.27)
+			)
+			(justify right bottom)
 		)
 	)
@@
 	)
 	(label "GRID3"
-		(at 81.6231 74.8562 0)
+		(at 250.063 62.4338 0)
 		(effects
 			(font
@@
 	)
 	(label "GRID4"
-		(at 81.6231 77.3962 0)
+		(at 250.063 64.9738 0)
 		(effects
 			(font
@@
 	)
 	(label "SEG3/KS3"
-		(at 81.6231 46.9749 0)
-		(effects
-			(font
-				(size 1.27 1.27)
-			)
-			(justify left bottom)
+		(at 194.183 52.2738 180)
+		(effects
+			(font
+				(size 1.27 1.27)
+			)
+			(justify right bottom)
 		)
 	)
 	(label "SEG6/KS6"
-		(at 81.6231 54.5949 0)
-		(effects
-			(font
-				(size 1.27 1.27)
-			)
-			(justify left bottom)
+		(at 194.183 59.8938 180)
+		(effects
+			(font
+				(size 1.27 1.27)
+			)
+			(justify right bottom)
 		)
 	)
 	(label "SEG2/KS2"
-		(at 81.6231 44.4349 0)
-		(effects
-			(font
-				(size 1.27 1.27)
-			)
-			(justify left bottom)
+		(at 194.183 49.7338 180)
+		(effects
+			(font
+				(size 1.27 1.27)
+			)
+			(justify right bottom)
 		)
 	)
 	(label "SEG1/KS1"
-		(at 81.6231 41.8949 0)
-		(effects
-			(font
-				(size 1.27 1.27)
-			)
-			(justify left bottom)
+		(at 194.183 47.1938 180)
+		(effects
+			(font
+				(size 1.27 1.27)
+			)
+			(justify right bottom)
 		)
 	)
@@
 	)
 	(label "SEG7/KS7"
-		(at 81.6231 57.1349 0)
-		(effects
-			(font
-				(size 1.27 1.27)
-			)
-			(justify left bottom)
+		(at 194.183 62.4338 180)
+		(effects
+			(font
+				(size 1.27 1.27)
+			)
+			(justify right bottom)
 		)
 	)
@@
 	)
 	(label "SEG5/KS5"
-		(at 81.6231 52.0549 0)
-		(effects
-			(font
-				(size 1.27 1.27)
-			)
-			(justify left bottom)
+		(at 194.183 57.3538 180)
+		(effects
+			(font
+				(size 1.27 1.27)
+			)
+			(justify right bottom)
 		)
 	)
 	(label "GRID2"
-		(at 81.6231 72.3162 0)
+		(at 250.063 59.8938 0)
 		(effects
 			(font
@@
 	)
 	(symbol
-		(lib_id "Connector:Conn_01x08_Pin")
-		(at 76.5431 49.5149 0)
-		(unit 1)
-		(exclude_from_sim no)
-		(in_bom yes)
-		(on_board yes)
-		(dnp no)
-		(property "Reference" "J3"
-			(at 78.4629 38.1679 0)
-			(effects
-				(font
-					(size 1.27 1.27)
-				)
-			)
-		)
-		(property "Value" "Conn_01x08_Pin"
-			(at 77.1781 39.9287 0)
-			(effects
-				(font
-					(size 1.27 1.27)
-				)
-				(hide yes)
-			)
-		)
-		(property "Footprint" "Connector_PinHeader_1.00mm:PinHeader_1x08_P1.00mm_Vertical"
-			(at 76.5431 49.5149 0)
-			(effects
-				(font
-					(size 1.27 1.27)
-				)
-				(hide yes)
-			)
-		)
-		(property "Datasheet" "~"
-			(at 76.5431 49.5149 0)
-			(effects
-				(font
-					(size 1.27 1.27)
-				)
-				(hide yes)
-			)
-		)
-		(property "Description" "Generic connector, single row, 01x08, script generated"
-			(at 76.5431 49.5149 0)
-			(effects
-				(font
-					(size 1.27 1.27)
-				)
-				(hide yes)
-			)
-		)
-		(pin "4"
-		)
-		(pin "5"
-		)
-		(pin "1"
-		)
-		(pin "2"
-		)
-		(pin "3"
-		)
-		(pin "6"
-		)
-		(pin "7"
-		)
-		(pin "8"
-		)
-		(instances
-			(project "seven segment"
-				(path "/f35e8fbd-20e2-4e8b-a22f-f96068be6e33"
-					(reference "J3")
-					(unit 1)
-				)
-			)
-		)
-	)
-	(symbol
 		(lib_id "power:GND1")
 		(at 112.0101 48.1744 180)
@@
 	)
 	(symbol
+		(lib_id "Display_Character:CC56-12EWA")
+		(at 222.123 54.8138 0)
+		(unit 1)
+		(exclude_from_sim no)
+		(in_bom yes)
+		(on_board yes)
+		(dnp no)
+		(fields_autoplaced yes)
+		(property "Reference" "U2"
+			(at 222.123 36.94 0)
+			(effects
+				(font
+					(size 1.27 1.27)
+				)
+			)
+		)
+		(property "Value" "CC56-12EWA"
+			(at 222.123 39.48 0)
+			(effects
+				(font
+					(size 1.27 1.27)
+				)
+			)
+		)
+		(property "Footprint" "Display_7Segment:CA56-12EWA"
+			(at 222.123 70.0538 0)
+			(effects
+				(font
+					(size 1.27 1.27)
+				)
+				(hide yes)
+			)
+		)
+		(property "Datasheet" "http://www.kingbrightusa.com/images/catalog/SPEC/CA56-12EWA.pdf"
+			(at 211.201 54.0518 0)
+			(effects
+				(font
+					(size 1.27 1.27)
+				)
+				(hide yes)
+			)
+		)
+		(property "Description" "4 digit 7 segment high efficiency red LED, common cathode"
+			(at 222.123 54.8138 0)
+			(effects
+				(font
+					(size 1.27 1.27)
+				)
+				(hide yes)
+			)
+		)
+		(pin "5"
+		)
+		(pin "3"
+		)
+		(pin "11"
+		)
+		(pin "12"
+		)
+		(pin "10"
+		)
+		(pin "2"
+		)
+		(pin "9"
+		)
+		(pin "4"
+		)
+		(pin "8"
+		)
+		(pin "7"
+		)
+		(pin "1"
+		)
+		(pin "6"
+		)
+		(instances
+			(project ""
+				(path "/f35e8fbd-20e2-4e8b-a22f-f96068be6e33"
+					(reference "U2")
+					(unit 1)
+				)
+			)
+		)
+	)
+	(symbol
 		(lib_id "power:GND1")
 		(at 171.5588 65.9544 0)
@@
 					(unit 1)
 				)
-			)
-		)
-	)
-	(symbol
-		(lib_id "Connector:Conn_01x04_Pin")
-		(at 76.5431 72.3162 0)
-		(unit 1)
-		(exclude_from_sim no)
-		(in_bom yes)
-		(on_board yes)
-		(dnp no)
-		(property "Reference" "J4"
-			(at 78.6953 66.4827 0)
-			(effects
-				(font
-					(size 1.27 1.27)
-				)
-			)
-		)
-		(property "Value" "Conn_01x04_Pin"
-			(at 77.1781 67.1765 0)
-			(effects
-				(font
-					(size 1.27 1.27)
-				)
-				(hide yes)
-			)
-		)
-		(property "Footprint" "Connector_PinHeader_2.54mm:PinHeader_1x04_P2.54mm_Vertical"
-			(at 76.5431 72.3162 0)
-			(effects
-				(font
-					(size 1.27 1.27)
-				)
-				(hide yes)
-			)
-		)
-		(property "Datasheet" "~"
-			(at 76.5431 72.3162 0)
-			(effects
-				(font
-					(size 1.27 1.27)
-				)
-				(hide yes)
-			)
-		)
-		(property "Description" "Generic connector, single row, 01x04, script generated"
-			(at 76.5431 72.3162 0)
-			(effects
-				(font
-					(size 1.27 1.27)
-				)
-				(hide yes)
-			)
-		)
-		(pin "2"
-		)
-		(pin "4"
-		)
-		(pin "1"
-		)
-		(pin "3"
-		)
-		(instances
-			(project "seven segment"
-				(path "/f35e8fbd-20e2-4e8b-a22f-f96068be6e33"
-					(reference "J4")
-					(unit 1)
-				)
