File: seven segment/seven segment.kicad_pcb (KiCad board)
At the start: 2 copper layers, 80.3 x 36.3 mm, 1 part

Commit message: -
Parts:
- added C1: 100nF, Capacitor_SMD:C_0603_1608Metric_Pad1.08x0.95mm_HandSolder, B.Cu at (101.2, 88.6)
- added C2: 10uF, Capacitor_SMD:C_0603_1608Metric_Pad1.08x0.95mm_HandSolder, B.Cu at (99.7, 88.6)
- added J1: Conn_01x04_Socket, Connector_JST:JST_EH_B4B-EH-A_1x04_P2.50mm_Vertical, F.Cu at (93.7, 86.5)
- added R1: 4.7k, Resistor_SMD:R_0603_1608Metric_Pad0.98x0.95mm_HandSolder, B.Cu at (101.2, 84.3)
- added R2: 4.7k, Resistor_SMD:R_0603_1608Metric_Pad0.98x0.95mm_HandSolder, B.Cu at (99.7, 84.3)
- added U1: CA56-12SRWA, Display_7Segment:CA56-12SRWA, F.Cu at (124.5, 97.8)
- added U2: TM1637, Footprint:SOP-20_L12.8-W7.5-P1.27-LS10.4-BL, B.Cu at (109.4, 90.1)
Routing:
- net /GRID3: track 0.00 -> 44.9 mm, vias 0 -> 1
- net /GRID4: track 0.00 -> 40.7 mm, vias 0 -> 1
- net /GRID2: track 0.00 -> 38.9 mm, vias 0 -> 1
- net /SEG7/KS7: track 0.00 -> 34.1 mm
- net /SEG8/KS8: track 0.00 -> 30.2 mm, vias 0 -> 1
- net /GRID1: track 0.00 -> 26.9 mm, vias 0 -> 1
- net /SEG3/KS3: track 0.00 -> 26.1 mm
- net /SEG2/KS2: track 0.00 -> 26.0 mm
- net /SEG6/KS6: track 0.00 -> 22.8 mm, vias 0 -> 1
- net /SEG4/KS4: track 0.00 -> 20.2 mm
- net +3.3VA: track 0.00 -> 19.0 mm
- net /DIO: track 0.00 -> 17.5 mm, vias 0 -> 1
- net /SEG5/KS5: track 0.00 -> 17.2 mm
- net /CLK: track 0.00 -> 14.8 mm, vias 0 -> 1
- net /SEG1/KS1: track 0.00 -> 14.4 mm
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- added copper zone on B.Cu, net GND1
- added copper zone on F.Cu, net GND1
Other:
- outline, holes or cut-outs redrawn
- board text added: "CLK"
- board text added: "DIO"
- board text added: "G"
- board text added: "V"
