File: Vendo_main_board/Vendo_main_board_ESP32/Vendo_main_board_ESP32.kicad_sch (KiCad schematic)
At the start: 100 parts, among them J1 Screw_Terminal_01x04, J10 Screw_Terminal_01x03, J11 Screw_Terminal_01x02, J12 Screw_Terminal_01x03, J2 Barrel_Jack_MountingPin, J3 Conn_01x05_Pin, J4 Conn_01x05_Pin, J6 Screw_Terminal_01x04, J7 Conn_01x04, J9 Conn_01x04_Pin, Q1 Q_NMOS_Depletion_GSD, Q2 Q_NMOS_Depletion_GSD, Q3 Q_NMOS_Depletion_GSD, Q4 Q_NMOS_Depletion_GSD, SW1 SW_Push, SW2 SW_Push, SW3 SW_Push, SW4 SW_Push, SW5 SW_Slide_DPDT, SW7 SW_Push, U1 AMS1117-3.3, U2 AP64350SP-13, U4 PC817, U5 TPL5010, U7 ESP32-WROOM-32

Commit message: - update schematic for esp32
- add esp32 , add wdt ,
- add rtc have problem on pin
Parts:
- removed C1, C4: 10uF, Capacitor_SMD:C_1206_3216Metric_Pad1.33x1.80mm_HandSolder, symbol Device:C
- removed C10: 3.3nF, Capacitor_SMD:C_0603_1608Metric, symbol Device:C
- removed C11: 56pF, Capacitor_SMD:C_0603_1608Metric, symbol Device:C
- removed C12, C13: 22uF, Capacitor_SMD:C_1210_3225Metric, symbol Device:C
- removed C26: 22uF, Capacitor_SMD:C_0603_1608Metric_Pad1.08x0.95mm_HandSolder, symbol Device:C_Polarized
- removed C7: 100nF, Capacitor_SMD:C_0603_1608Metric_Pad1.08x0.95mm_HandSolder, symbol Device:C
- removed J7: Conn_01x04, Connector_JST:JST_EH_B4B-EH-A_1x04_P2.50mm_Vertical, symbol Connector_Generic:Conn_01x04
- removed L1: 6.8uH, InnovKits:IND-SMD_L11.5-W10.0_FXL1040, symbol pspice:INDUCTOR
- removed R1: 200k, Resistor_SMD:R_0603_1608Metric_Pad0.98x0.95mm_HandSolder, symbol Device:R
- removed R31: 10K, Resistor_SMD:R_0603_1608Metric_Pad0.98x0.95mm_HandSolder, symbol Device:R
- removed R5: 14k, Resistor_SMD:R_0603_1608Metric_Pad0.98x0.95mm_HandSolder, symbol Device:R
- removed R6: 28k, Resistor_SMD:R_0603_1608Metric_Pad0.98x0.95mm_HandSolder, symbol Device:R
- removed R7: 147k, Resistor_SMD:R_0603_1608Metric_Pad0.98x0.95mm_HandSolder, symbol Device:R
- removed U2: AP64350SP-13, InnovKits:AP64350SP-13-L, symbol adp650:AP64350SP-13
- added BT1: Battery_Cell, InnovKits:BAT-TH_CR2032-BS-6-1, symbol Device:Battery_Cell
- added C1, C4: 4.7uF/50V, Capacitor_SMD:C_1206_3216Metric, symbol tps:C
- added C10: 0.01uF, Capacitor_SMD:C_0603_1608Metric, symbol tps:C
- added C11: 0.1uF/50V, Capacitor_SMD:C_0603_1608Metric, symbol tps:C
- added C12: 68pF, Capacitor_SMD:C_0603_1608Metric, symbol tps:C
- added C13: 8200pF, Capacitor_SMD:C_0603_1608Metric, symbol tps:C
- added C14: 22uF, Capacitor_SMD:C_0603_1608Metric_Pad1.08x0.95mm_HandSolder, symbol Device:C_Polarized
- added C15: 10uF, Capacitor_SMD:C_0603_1608Metric_Pad1.08x0.95mm_HandSolder, symbol Device:C
- added C16: 100nF, Capacitor_SMD:C_0603_1608Metric_Pad1.08x0.95mm_HandSolder, symbol Device:C
- added C25, C26: 22uF/16V, Capacitor_SMD:C_1210_3225Metric, symbol tps:C
- added C7: 0.01uF/50V, Capacitor_SMD:C_0603_1608Metric, symbol tps:C
- added D1: SS34, Diode_SMD:D_SMA, symbol tps:D_Schottky
- added J7: FTDI, Connector_PinHeader_2.54mm:PinHeader_1x04_P2.54mm_Vertical, symbol Connector:Conn_01x04_Pin
- added L1: 10uH, InnovKits:IND-SMD_L11.5-W10.0_FXL1040, symbol tps:L
- added R1: 332k, Resistor_SMD:R_0603_1608Metric, symbol tps:R
- added R28: 10.5k, Resistor_SMD:R_0603_1608Metric, symbol tps:R
- added R31: 2.00k, Resistor_SMD:R_0603_1608Metric, symbol tps:R
- added R5: 68.1k, Resistor_SMD:R_0603_1608Metric, symbol tps:R
- added R6: 28.0k, Resistor_SMD:R_0603_1608Metric, symbol tps:R
- added R7: 0R, Resistor_SMD:R_0603_1608Metric, symbol tps:R
- added R8: 10K, Resistor_SMD:R_0603_1608Metric_Pad0.98x0.95mm_HandSolder, symbol Device:R
- added U2: TPS54331D, Package_SO:SOIC-8_3.9x4.9mm_P1.27mm, symbol tps:TPS54331D
- added U6: SOLA-IC SLM1302, Package_SO:SOIC-8_3.9x4.9mm_P1.27mm, symbol Timer_RTC:DS1302ZN+
- added Y1: Crystal, InnovKits:OSC-SMD_L3.2-W1.5, symbol Device:Crystal
Connections:
- net +12V: now also C1.1, C4.1, C7.1, R1.1, U2.2 (VIN)
- net +3.3V: now also C14.1, C15.1, C16.1, R8.1, U6.1 (VCC2)
- net +5V: now also C25.1, C26.1, J7.1 (Pin_1), L1.2, R7.1
- net ESP_I0: now also R8.2
- net ESP_RX: now also J7.3 (Pin_3)
- net ESP_TX: now also J7.2 (Pin_2)
- net GND: now also BT1.2 (-), C1.2, C10.2, C12.2, C14.2, C15.2, C16.2, C25.2, C26.2, C4.2, C7.2, D1.2 (A), J7.4 (Pin_4), R31.2, R5.2, R6.2, U2.7 (GND), U6.4 (GND)
- new net: BT1.1 (+), U6.8 (VCC1)
- new net: U6.3 (X2), Y1.1
- new net: U6.2 (X1), Y1.2
- new net BOOT: C11.1, U2.1 (BOOT)
- new net COMP: C12.1, C13.1, U2.6 (COMP)
- new net CZ: C13.2, R6.1
- new net EN: R1.2, R5.1, U2.3 (EN)
- new net FB: R28.2, R31.1, U2.5 (VSENSE)
- new net FB_TOP: R28.1, R7.2
- new net RTC_CE: U6.5 (CE)
- new net RTC_CLK: U6.7 (SCLK)
- new net RTC_DAT: U6.6 (I/O)
- new net SS: C10.1, U2.4 (SS)
- new net SW: C11.2, D1.1 (K), L1.1, U2.8 (PH)
Other:
- note added: "REAL-TIME CLOCK"
- moved on the sheet: BZ1, C17, C2, C27, C28, C29, C3, C5, C6, C8, C9, D3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
