File: Vendo_main_board/Vendo_main_board_ESP32/Vendo_main_board_ESP32/Vendo_main_board_ESP32.kicad_sch (KiCad schematic)
At the start: 106 parts, among them J1 Screw_Terminal_01x04, J10 Screw_Terminal_01x03, J11 Screw_Terminal_01x02, J12 Screw_Terminal_01x03, J2 Barrel_Jack_MountingPin, J3 Conn_01x05_Pin, J4 Conn_01x05_Pin, J6 Screw_Terminal_01x04, J7 FTDI, J9 Conn_01x04_Pin, Q1 Q_NMOS_Depletion_GSD, Q2 Q_NMOS_Depletion_GSD, Q3 Q_NMOS_Depletion_GSD, Q4 Q_NMOS_Depletion_GSD, SW1 SW_Push, SW2 SW_Push, SW3 SW_Push, SW5 SW_Slide_DPDT, SW7 SW_Push, U1 AMS1117-3.3, U2 TPS54331D, U4 PC817, U5 TPL5010, U6 SOLA-IC SLM1302, U7 ESP32-WROOM-32, Y1 Crystal

Commit message: stm32 and esp32 version edit
stm32 ver solid gnd plane to buck conv, adjust buttons to smd , btn1 to 3 and reset
esp32 version adjust slave conn by 1mm far away on the sma hole, adjust button 1 ,2 and reset.
Parts:
- SW1, SW2, SW3: footprint Button_Switch_THT:SW_PUSH_6mm_H5mm -> Button_Switch_SMD:SW_SPST_PTS645
Changed lines of the file:
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@@
 			)
 		)
-		(property "Footprint" "Button_Switch_THT:SW_PUSH_6mm_H5mm"
+		(property "Footprint" "Button_Switch_SMD:SW_SPST_PTS645"
 			(at 344.6119 232.41 0)
 			(effects
@@
 			)
 		)
-		(property "Footprint" "Button_Switch_THT:SW_PUSH_6mm_H5mm"
+		(property "Footprint" "Button_Switch_SMD:SW_SPST_PTS645"
 			(at 406.297 313.6996 0)
 			(effects
@@
 			)
 		)
-		(property "Footprint" "Button_Switch_THT:SW_PUSH_6mm_H5mm"
+		(property "Footprint" "Button_Switch_SMD:SW_SPST_PTS645"
 			(at 375.817 313.6996 0)
 			(effects
