File: Vendo_board_jigg/Vendo_board_jigg.kicad_pcb (KiCad board)
At the start: 2 copper layers, 60 x 100 mm, 64 parts, among them J1 Screw_Terminal_01x04, J10 Screw_Terminal_01x03, J12 Screw_Terminal_01x03, J2 Barrel_Jack_MountingPin, J3 Conn_01x05_Pin, J4 Conn_01x05_Pin, J6 Screw_Terminal_01x04, J7 FTDI, J9 Conn_01x04_Pin, Q3 Q_NMOS_Depletion_GSD, SW1 SW_Push, SW7 SW_Push, U1 AMS1117-3.3, U4 PC817, U7 ESP32-WROOM-32

Commit message: -vendo jigg
-added placement for pcb of the vendo jigg
Parts:
- removed the H4 at (202.6, 123.1)
- removed JP7: Jumper_3_Open, Connector_PinHeader_2.54mm:PinHeader_1x03_P2.54mm_Vertical
- removed JP8: SolderJumper_2_Open, Jumper:SolderJumper-2_P1.3mm_Open_RoundedPad1.0x1.5mm
- removed Q3: Q_NMOS_Depletion_GSD, Package_TO_SOT_SMD:SOT-23-3
- removed R22, R24, R25: 1K, Resistor_SMD:R_0603_1608Metric_Pad0.98x0.95mm_HandSolder
- removed R23, R26: 1k, Resistor_SMD:R_0603_1608Metric_Pad0.98x0.95mm_HandSolder
- removed U4: PC817, InnovKits:APC-817xx-SL_AMB
- removed kibuzzard-6A0C4EC9: G***, kibuzzard-6A0C4EC9
- removed kibuzzard-6A0C5F1E: G***, kibuzzard-6A0C5F1E
- removed kibuzzard-6A563CE9: G***, kibuzzard-6A563CE9
- added C1: 0.1uF, Capacitor_SMD:C_0805_2012Metric_Pad1.18x1.45mm_HandSolder, F.Cu at (265.4, 82.0)
- added C10: 10uF, Capacitor_SMD:C_0805_2012Metric_Pad1.18x1.45mm_HandSolder, F.Cu at (259.2, 71.1)
- added C4: 0.1uF, Capacitor_SMD:C_0805_2012Metric_Pad1.18x1.45mm_HandSolder, F.Cu at (265.2, 71.1)
- added C7: 100nF, Capacitor_SMD:C_0603_1608Metric_Pad1.08x0.95mm_HandSolder, F.Cu at (233.6, 114.4)
- added D1: LED, LED_SMD:LED_0805_2012Metric_Pad1.15x1.40mm_HandSolder, F.Cu at (267.0, 104.0)
- added D2: LED, LED_SMD:LED_0805_2012Metric_Pad1.15x1.40mm_HandSolder, F.Cu at (267.0, 102.0)
- added J11: Conn_01x04_Pin, Connector_JST:JST_EH_B4B-EH-A_1x04_P2.50mm_Vertical, F.Cu at (267.7, 64.3)
- added J5: Barrel_Jack_MountingPin, Connector_BarrelJack:BarrelJack_GCT_DCJ200-10-A_Horizontal, F.Cu at (265.4, 39.1)
- added J8: Screw_Terminal_01x03, TerminalBlock:TerminalBlock_Xinya_XY308-2.54-3P_1x03_P2.54mm_Horizontal, F.Cu at (261.9, 122.3)
- added JP14: SolderJumper_2_Open, Connector_PinHeader_2.54mm:PinHeader_1x02_P2.54mm_Vertical, F.Cu at (268.6, 98.3)
- added Q5: BSS138, Package_TO_SOT_SMD:SOT-23, F.Cu at (262.1, 71.2)
- added Q6: BSS138, Package_TO_SOT_SMD:SOT-23, F.Cu at (268.2, 71.2)
- added R1: 5.1k, Resistor_SMD:R_0603_1608Metric_Pad0.98x0.95mm_HandSolder, F.Cu at (262.2, 87.3)
- added R11: 100K, Resistor_SMD:R_0603_1608Metric_Pad0.98x0.95mm_HandSolder, F.Cu at (232.0, 114.4)
- added R13: 4.7K, Resistor_SMD:R_0603_1608Metric_Pad0.98x0.95mm_HandSolder, F.Cu at (213.8, 42.5)
- added R14: 10K, Resistor_SMD:R_0603_1608Metric_Pad0.98x0.95mm_HandSolder, F.Cu at (203.7, 104.8)
- added R15: 10K, Resistor_SMD:R_0603_1608Metric_Pad0.98x0.95mm_HandSolder, F.Cu at (203.7, 108.2)
- added R16: 10K, Resistor_SMD:R_0603_1608Metric_Pad0.98x0.95mm_HandSolder, F.Cu at (217.2, 42.5)
- added R17: 10K, Resistor_SMD:R_0603_1608Metric_Pad0.98x0.95mm_HandSolder, F.Cu at (223.4, 42.5)
- added R18: 4.7K, Resistor_SMD:R_0603_1608Metric_Pad0.98x0.95mm_HandSolder, F.Cu at (200.7, 104.8)
- added R19: 4.7K, Resistor_SMD:R_0603_1608Metric_Pad0.98x0.95mm_HandSolder, F.Cu at (226.8, 42.5)
- added R20: 1K, Resistor_SMD:R_0603_1608Metric_Pad0.98x0.95mm_HandSolder, F.Cu at (217.7, 115.9)
- added R27: 10K, Resistor_SMD:R_0603_1608Metric_Pad0.98x0.95mm_HandSolder, F.Cu at (235.4, 101.6)
- added R28: 10K, Resistor_SMD:R_0603_1608Metric_Pad0.98x0.95mm_HandSolder, F.Cu at (200.7, 108.2)
- added R4: 4.7K, Resistor_SMD:R_0603_1608Metric_Pad0.98x0.95mm_HandSolder, F.Cu at (236.9, 101.5)
- added R5: 33K, Resistor_SMD:R_0603_1608Metric_Pad0.98x0.95mm_HandSolder, F.Cu at (206.5, 104.8)
- added R6: 1K, Resistor_SMD:R_0603_1608Metric_Pad0.98x0.95mm_HandSolder, F.Cu at (263.2, 104.2)
- added R7: 1K, Resistor_SMD:R_0603_1608Metric_Pad0.98x0.95mm_HandSolder, F.Cu at (263.2, 101.9)
- added R9: 10K, Resistor_SMD:R_0603_1608Metric_Pad0.98x0.95mm_HandSolder, F.Cu at (206.5, 108.2)
- added U2: CH340C, Package_SO:SOP-16_3.9x9.9mm_P1.27mm, F.Cu at (265.0, 77.1)
- added USB1: TYPE C TYPE C, InnovKits:USB-C-SMD_TYPE-C16PIN, F.Cu at (267.2, 90.0)
- BZ1: value Buzzer -> BUZZER_PORT
- JP6: value SolderJumper_3_Open -> SolderJumper_2_Open; footprint Jumper:SolderJumper-3_P1.3mm_Open_Pad1.0x1.5mm_NumberLabels -> Connector_PinHeader_2.54mm:PinHeader_1x02_P2.54mm_Vertical; moved to F.Cu
- R10: value 1K -> 5.1k
- R21: value 10K -> 1K; footprint Resistor_SMD:R_0805_2012Metric_Pad1.20x1.40mm_HandSolder -> Resistor_SMD:R_0603_1608Metric_Pad0.98x0.95mm_HandSolder
- moved R10 53.6 mm to (262.3, 92.2), turned to -90 degrees
- moved JP6 22.7 mm to (266.1, 49.0), turned to 90 degrees
- moved R21 17.9 mm to (219.2, 115.9), turned to -90 degrees
- moved SW1 12.9 mm to (265.2, 110.6), turned to 180 degrees
- moved kibuzzard-6A0C5003 12.2 mm to (265.3, 41.5)
- moved C17 11.8 mm to (259.3, 109.0), turned to -90 degrees
- moved C5 11.1 mm to (218.6, 63.0)
- moved C9 11.1 mm to (224.4, 63.2)
- moved C3 11.1 mm to (226.2, 63.0)
- moved C8 11.1 mm to (220.4, 63.2)
- moved C2 11.1 mm to (228.2, 63.4)
- moved C6 11.1 mm to (222.4, 63.4)
- moved U1 11.1 mm to (224.0, 56.5)
- moved kibuzzard-6A0C536D 9.26 mm to (265.1, 115.0), turned to 0 degrees
- moved R12 7.00 mm to (259.3, 112.4), turned to 90 degrees
Connections:
- J1 pad 1: USER_BTN -> USER_BTN_TEST
- J1 pad 3: Net-(J1-Pin_3) -> unconnected-(J1-Pin_3-Pad3)
- J1 pad 4: Net-(J1-Pin_4) -> USER_LED_TEST
- J10 pad 3: +12V -> Net-(J10-Pin_3)
- J12 pad 1: RLY_NC -> Net-(J12-Pin_1)
- J12 pad 2: RLY_COM -> Net-(J12-Pin_2)
- J12 pad 3: RLY_NO -> Net-(J12-Pin_3)
- J6 pad 1: Net-(J6-Pin_1) -> unconnected-(J6-Pin_1-Pad1)
- J6 pad 2: AUX_1 -> AUX_1_TEST
- J6 pad 3: AUX_2 -> AUX_2_TEST
- J7 pad 2: ESP_TX -> ESP_JIGG_TX
- J7 pad 3: ESP_RX -> ESP_JIGG_RX
- J9 pad 1: Net-(J9-Pin_1) -> Net-(J11-Pin_1)
- J9 pad 2: SEG_CLK -> Net-(J11-Pin_2)
- J9 pad 3: SEG_DIO -> Net-(J11-Pin_3)
- JP10 pad 1: GND -> unconnected-(JP10-A-Pad1)
- JP3 pad 1: Net-(J1-Pin_3) -> Net-(JP3-A)
- JP4 pad 1: Net-(J1-Pin_3) -> Net-(JP4-A)
- JP5 pad 1: Net-(J1-Pin_3) -> Net-(JP5-A)
- JP6 pad 1: +3.3V -> Net-(J12-Pin_2)
- JP6 pad 2: Net-(J9-Pin_1) -> +3.3V
- R10 pad 1: +3.3V -> Net-(USB1-CC1)
- R10 pad 2: USER_BTN -> GND
- R21 pad 1: COIN_EN -> +3.3V
- R21 pad 2: GND -> AUX_2_TEST
- U7 pad 10: RTC_CE -> RELAY_NC_TEST
- U7 pad 11: RTC_CLK -> RELAY_NO_TEST
- U7 pad 12: BUZZER -> BUZZER_TEST
- U7 pad 13: SEG_DIO -> AUX_2_TEST
- U7 pad 14: COIN_EN -> unconnected-(U7-IO12-Pad14)
- U7 pad 16: SEG_CLK -> AUX_1_TEST
- U7 pad 23: DBG_LED_B -> I2C_INT
- U7 pad 24: WDT_DONE -> unconnected-(U7-IO2-Pad24)
- U7 pad 26: RTC_DAT -> unconnected-(U7-IO4-Pad26)
- U7 pad 27: I2C_INT -> ESP_JIGG_TX
- U7 pad 28: COIN_IN -> ESP_JIGG_RX
- U7 pad 29: I2C_CONFG -> unconnected-(U7-IO5-Pad29)
- U7 pad 30: USER_BTN -> USER_BTN_TEST
- U7 pad 31: RLY_DRV -> I2C_CONFG
- U7 pad 37: USER_LED -> USER_LED_TEST
- U7 pad 6: BTN_MODE_1 -> unconnected-(U7-IO34-Pad6)
- U7 pad 7: BTN_MODE_2 -> unconnected-(U7-IO35-Pad7)
- U7 pad 8: AUX_1 -> 12V_ADC
- U7 pad 9: AUX_2 -> 5V_ADC
Other:
- board size 60 x 100 mm -> 72.5 x 100 mm
- board text added: "A1"
- board text added: "A2"
- board text added: "COIN SLOT"
- board text added: "COM 3.3V"
- board text added: "LCD"
- board text removed: "DESIGNED AND MANUFACTURED BY:"
- board text removed: "ENGINEERING SMARTER VENDING SOLUTIONS"
- board text removed: "VENDO BOARD V1.0"
- board text removed: "VendoLabsPH"
