File: Vendo_board_jigg/Vendo_board_jigg.kicad_sch (KiCad schematic)
At the start: 73 parts, among them J1 Screw_Terminal_01x04, J10 Screw_Terminal_01x03, J11 Conn_01x04_Pin, J12 Screw_Terminal_01x03, J2 Barrel_Jack_MountingPin, J3 Conn_01x05_Pin, J4 Conn_01x05_Pin, J5 Barrel_Jack_MountingPin, J6 Screw_Terminal_01x04, J7 FTDI, J8 Screw_Terminal_01x03, J9 Conn_01x04_Pin, Q5 BSS138, Q6 BSS138, SW1 SW_Push, SW7 SW_Push, U1 AMS1117-3.3, U2 CH340C, U7 ESP32-WROOM-32

Commit message: -vendo jigg
-added placement for pcb of the vendo jigg
Parts:
- JP14: footprint (none) -> Connector_PinHeader_2.54mm:PinHeader_1x02_P2.54mm_Vertical
- USB1: value ~ -> TYPE C TYPE C; footprint tanimoji:USB-C-SMD_TYPE-C16PIN -> InnovKits:USB-C-SMD_TYPE-C16PIN
- renumbered C4 to C10, R1 to R10
